File: microconsole_hardware/mc_hw/mc_hw.kicad_pcb (KiCad board)
At the start: 2 copper layers, 25 parts, among them SW1 DPAD - UP, SW10 START, SW11 L1, SW12 R1, SW13 L2, SW14 R2, SW16 Joystick, SW17 Joystick, SW2 DPAD - DOWN, SW3 DPAD - LEFT, SW4 DPAD - RIGHT, SW5 A, SW6 B, SW7 X, SW8 Y, SW9 SELECT, U1 CR2013-MI2120, U2 MAX98357A, U3 MCP23017x-x-SO

Commit message: quick fix
Parts:
- A1: moved to B.Cu
- turned A1 to 180 degrees
Connections:
- net GPIO3 / MCP|ADC SCK renamed GPIO3 / MCP|ADC SCL
- net GPIO4 / ILI MISO renamed GPIO4 / LCD MISO
- net GPIO5 / ILI CS renamed GPIO5 / LCD CS
- net GPIO6 / ILI SCK renamed GPIO6 / LCD SCK
- net GPIO7 / ILI MOSI renamed GPIO7 / LCD MOSI
- net GPIO8 / ILI RESET renamed GPIO8 / LCD RESET
- net GPIO9 / ILI DC renamed GPIO9 / LCD DC
- U3 pad 9: VBUS -> 3v3

Commit message: Update mc_hw.kicad_pcb
Parts:
- added C1: 100nF, Capacitor_SMD:C_0603_1608Metric_Pad1.08x0.95mm_HandSolder, F.Cu at (57.5, 96.8)
- added C10: 10uF, Capacitor_SMD:C_0805_2012Metric_Pad1.18x1.45mm_HandSolder, F.Cu at (52.9, 106.0)
- added C11: 10uF, Capacitor_SMD:C_0805_2012Metric_Pad1.18x1.45mm_HandSolder, F.Cu at (52.9, 109.0)
- added C12: 100nF, Capacitor_SMD:C_0603_1608Metric_Pad1.08x0.95mm_HandSolder, F.Cu at (57.5, 111.8)
- added C13: 10uF, Capacitor_SMD:C_0805_2012Metric_Pad1.18x1.45mm_HandSolder, F.Cu at (52.9, 112.1)
- added C2: 100nF, Capacitor_SMD:C_0603_1608Metric_Pad1.08x0.95mm_HandSolder, F.Cu at (57.5, 99.3)
- added C3: 100nF, Capacitor_SMD:C_0603_1608Metric_Pad1.08x0.95mm_HandSolder, F.Cu at (57.5, 101.8)
- added C4: 10uF, Capacitor_SMD:C_0805_2012Metric_Pad1.18x1.45mm_HandSolder, F.Cu at (52.9, 97.0)
- added C5: 100nF, Capacitor_SMD:C_0603_1608Metric_Pad1.08x0.95mm_HandSolder, F.Cu at (57.5, 104.3)
- added C6: 100nF, Capacitor_SMD:C_0603_1608Metric_Pad1.08x0.95mm_HandSolder, F.Cu at (57.5, 106.8)
- added C7: 100nF, Capacitor_SMD:C_0603_1608Metric_Pad1.08x0.95mm_HandSolder, F.Cu at (57.5, 109.3)
- added C8: 10uF, Capacitor_SMD:C_0805_2012Metric_Pad1.18x1.45mm_HandSolder, F.Cu at (52.9, 100.0)
- added C9: 10uF, Capacitor_SMD:C_0805_2012Metric_Pad1.18x1.45mm_HandSolder, F.Cu at (52.9, 103.0)
- added R3: 10k, PCM_SparkFun-Resistor:R_0603_1608Metric, F.Cu at (61.7, 96.8)
- U1: value CR2013-MI2120 -> ILI9341 / ST7796S SPI LCD
- moved SW3 15.0 mm to (70.0, 120.0)
- moved SW1 13.0 mm to (80.0, 130.0), turned to 90 degrees
- moved SW2 10.9 mm to (80.0, 110.0), turned to 90 degrees
- moved SW4 9.01 mm to (90.0, 120.0)
Connections:
- A1 pad 4: Net-(A1-GPIO2) -> GPIO2 / MCP|ADC SDA
- A1 pad 5: Net-(A1-GPIO3) -> GPIO3 / MCP|ADC SCL
- R1 pad 1: GPIO2 / MCP|ADC SDA -> 3v3
- R1 pad 2: Net-(A1-GPIO2) -> GPIO2 / MCP|ADC SDA
- R2 pad 1: GPIO3 / MCP|ADC SCL -> 3v3
- R2 pad 2: Net-(A1-GPIO3) -> GPIO3 / MCP|ADC SCL
- U2 pad 17: unconnected-(U2-PAD-Pad17) -> GND
- U2 pad 4: unconnected-(U2-~{SD_MODE}-Pad4) -> VBUS
- U3 pad 18: unconnected-(U3-~{RESET}-Pad18) -> MCP RESET
Other:
- board outline added: 6.3 x 6.3 mm

Commit message: update symbols and libraries
Parts:
- C1, C10, C11, C12, C13, C2, C3, C4, C5, C6, C7, C8, C9, LS1, R1, R2, R3, U2, U3, U4: moved to B.Cu
- U1: footprint Display:CR2013-MI2120 -> microconsole:TFT
- moved C9 127.1 mm to (180.0, 105.0)
- moved C2 122.5 mm to (180.0, 100.0), turned to 180 degrees
- moved RV1 110.1 mm to (120.0, 148.1)
- moved C1 101.3 mm to (149.1, 140.0), turned to 180 degrees
- moved R3 98.7 mm to (160.0, 105.0), turned to -90 degrees
- moved C11 97.6 mm to (132.5, 52.5), turned to 90 degrees
- moved C6 96.7 mm to (137.5, 52.5), turned to -90 degrees
- moved C4 92.2 mm to (145.0, 92.5), turned to -90 degrees
- moved C7 91.6 mm to (147.5, 92.5), turned to -90 degrees
- moved C8 88.7 mm to (141.0, 90.0)
- moved C13 84.3 mm to (112.5, 52.5), turned to -90 degrees
- moved C3 84.1 mm to (141.0, 92.5)
- moved C12 77.6 mm to (107.5, 52.5), turned to 90 degrees
- moved C10 61.4 mm to (101.5, 68.5), turned to 90 degrees
- moved C5 53.4 mm to (97.2, 68.6), turned to -90 degrees
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Connections:
- C5 pad 1: 3v3 -> VBUS
- U3 pad 4: unconnected-(U3-GPB3-Pad4) -> MCP GPB3 / L1
- U3 pad 5: unconnected-(U3-GPB4-Pad5) -> MCP GPB4 / R1
- U3 pad 6: unconnected-(U3-GPB5-Pad6) -> MCP GPB5 / L2
- U3 pad 7: unconnected-(U3-GPB6-Pad7) -> MCP GPB6 / R2
Other:
- board size 6.3 x 6.3 mm -> 200 x 130 mm

Commit message: update hardware
Parts:
- U1: footprint microconsole:TFT -> microconsole_hardware:TFT
- U4: footprint microconsole:PCB0029_Footprint -> microconsole_hardware:PCB0029_Footprint
Changed lines of the file:
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@@
 		)
 	)
-	(footprint "microconsole:TFT"
+	(footprint "microconsole_hardware:TFT"
 		(layer "F.Cu")
 		(at 147.150001 105.175)
@@
 		(embedded_fonts no)
 		(model "${KICAD10_3DMODEL_DIR}/Display.3dshapes/CR2013-MI2120.step"
-			(hide yes)
 			(offset
 				(xyz 0 0 0)
@@
 			)
 		)
-		(property "Datasheet" "~"
+		(property "Datasheet" ""
 			(at 0 0 90)
 			(layer "B.Fab")
@@
 			)
 		)
-		(property "Description" "100nF volume ADC noise filter"
+		(property "Description" "Unpolarized capacitor"
 			(at 0 0 90)
 			(layer "B.Fab")
@@
 			(roundrect_rratio 0.212766)
 			(net "GND")
-			(pinfunction "~_1")
 			(pintype "passive")
 		)
@@
 			(roundrect_rratio 0.212766)
 			(net "VBUS")
-			(pinfunction "~_2")
 			(pintype "passive")
 		)
@@
 			)
 		)
-		(property "Datasheet" "~"
+		(property "Datasheet" ""
 			(at 0 0 0)
 			(layer "B.Fab")
@@
 			)
 		)
-		(property "Description" "100nF volume ADC noise filter"
+		(property "Description" "Unpolarized capacitor"
 			(at 0 0 0)
 			(layer "B.Fab")
@@
 			(roundrect_rratio 0.212766)
 			(net "GND")
-			(pinfunction "~_1")
 			(pintype "passive")
 		)
@@
 			(roundrect_rratio 0.212766)
 			(net "VBUS")
-			(pinfunction "~_2")
 			(pintype "passive")
 		)
@@
 			)
 		)
-		(property "Datasheet" "~"
+		(property "Datasheet" ""
 			(at 0 0 90)
 			(layer "B.Fab")
@@
 			)
 		)
-		(property "Description" "100nF volume ADC noise filter"
+		(property "Description" "Unpolarized capacitor"
 			(at 0 0 90)
 			(layer "B.Fab")
@@
 			(roundrect_rratio 0.25)
 			(net "3v3")
-			(pinfunction "~_1")
 			(pintype "passive")
 		)
@@
 			(roundrect_rratio 0.25)
 			(net "GND")
-			(pinfunction "~_2")
 			(pintype "passive")
 		)
@@
 			)
 		)
-		(property "Datasheet" "~"
+		(property "Datasheet" ""
 			(at 0 0 0)
 			(layer "B.Fab")
@@
 			)
 		)
-		(property "Description" "100nF volume ADC noise filter"
+		(property "Description" "Unpolarized capacitor"
 			(at 0 0 0)
 			(layer "B.Fab")
@@
 			(roundrect_rratio 0.212766)
 			(net "GND")
-			(pinfunction "~_1")
 			(pintype "passive")
 		)
@@
 			(roundrect_rratio 0.212766)
 			(net "3v3")
-			(pinfunction "~_2")
 			(pintype "passive")
 		)
@@
 			)
 		)
-		(property "Datasheet" "~"
+		(property "Datasheet" ""
 			(at 0 0 90)
 			(layer "B.Fab")
@@
 			)
 		)
-		(property "Description" "100nF volume ADC noise filter"
+		(property "Description" "Unpolarized capacitor"
 			(at 0 0 90)
 			(layer "B.Fab")
@@
 			(roundrect_rratio 0.212766)
 			(net "GND")
-			(pinfunction "~_1")
 			(pintype "passive")
 		)
@@
 			(roundrect_rratio 0.212766)
 			(net "3v3")
-			(pinfunction "~_2")
 			(pintype "passive")
 		)
@@
 			)
 		)
-		(property "Datasheet" "~"
+		(property "Datasheet" ""
 			(at 0 0 0)
 			(layer "B.Fab")
@@
 			)
 		)
-		(property "Description" "100nF volume ADC noise filter"
+		(property "Description" "Unpolarized capacitor"
 			(at 0 0 0)
 			(layer "B.Fab")
@@
 			(roundrect_rratio 0.25)
 			(net "3v3")
-			(pinfunction "~_1")
 			(pintype "passive")
 		)
@@
 			(roundrect_rratio 0.25)
 			(net "GND")
-			(pinfunction "~_2")
 			(pintype "passive")
 		)
@@
 			)
 		)
-		(property "Datasheet" "~"
+		(property "Datasheet" ""
 			(at 0 0 90)
 			(layer "B.Fab")
@@
 			)
 		)
-		(property "Description" "100nF volume ADC noise filter"
+		(property "Description" "Unpolarized capacitor"
 			(at 0 0 90)
 			(layer "B.Fab")
@@
 			(roundrect_rratio 0.25)
 			(net "VBUS")
-			(pinfunction "~_1")
 			(pintype "passive")
 		)
@@
 			(roundrect_rratio 0.25)
 			(net "GND")
-			(pinfunction "~_2")
 			(pintype "passive")
 		)
@@
 			)
 		)
-		(property "Datasheet" "~"
+		(property "Datasheet" ""
 			(at 0 0 90)
 			(layer "B.Fab")
@@
 			)
 		)
-		(property "Description" "100nF volume ADC noise filter"
+		(property "Description" "Unpolarized capacitor"
 			(at 0 0 90)
 			(layer "B.Fab")
@@
 			(roundrect_rratio 0.25)
 			(net "GND")
-			(pinfunction "~_1")
 			(pintype "passive")
 		)
@@
 			(roundrect_rratio 0.25)
 			(net "VBUS")
-			(pinfunction "~_2")
 			(pintype "passive")
 		)
@@
 			)
 		)
-		(property "Datasheet" "~"
+		(property "Datasheet" ""
 			(at 0 0 90)
 			(layer "B.Fab")
@@
 			)
 		)
-		(property "Description" "100nF volume ADC noise filter"
+		(property "Description" "Unpolarized capacitor"
 			(at 0 0 90)
 			(layer "B.Fab")
@@
 			(roundrect_rratio 0.25)
 			(net "VBUS")
-			(pinfunction "~_1")
 			(pintype "passive")
 		)
@@
 			(roundrect_rratio 0.25)
 			(net "GND")
-			(pinfunction "~_2")
 			(pintype "passive")
 		)
@@
 			)
 		)
-		(property "Datasheet" "~"
+		(property "Datasheet" ""
 			(at 0 0 0)
 			(layer "B.Fab")
@@
 			)
 		)
-		(property "Description" "100nF volume ADC noise filter"
+		(property "Description" "Unpolarized capacitor"
 			(at 0 0 0)
 			(layer "B.Fab")
@@
 			(roundrect_rratio 0.25)
 			(net "AGND")
-			(pinfunction "~_1")
 			(pintype "passive")
 		)
@@
 			(roundrect_rratio 0.25)
 			(net "GPIO28 {slash} VOLUME POT")
-			(pinfunction "~_2")
 			(pintype "passive")
 		)
@@
 			(net "GND")
 			(pinfunction "PAD_17")
-			(pintype "unspecified")
+			(pintype "power_in")
 			(zone_connect 2)
 		)
@@
 			(roundrect_rratio 0.25)
 			(net "GPIO3 {slash} MCP|ADC SCL")
-			(pinfunction "SCL_12")
+			(pinfunction "SCK_12")
 			(pintype "input")
 		)
@@
 			)
 		)
-		(property "Datasheet" "~"
+		(property "Datasheet" ""
 			(at 0 0 90)
 			(layer "B.Fab")
@@
 			)
 		)
-		(property "Description" "100nF volume ADC noise filter"
+		(property "Description" "Unpolarized capacitor"
 			(at 0 0 90)
 			(layer "B.Fab")
@@
 			(roundrect_rratio 0.212766)
 			(net "GND")
-			(pinfunction "~_1")
 			(pintype "passive")
 		)
@@
 			(roundrect_rratio 0.212766)
 			(net "VBUS")
-			(pinfunction "~_2")
 			(pintype "passive")
 		)
@@
 			)
 		)
-		(property "Datasheet" "~"
+		(property "Datasheet" ""
 			(at 0 0 0)
 			(layer "B.Fab")
@@
 			)
 		)
-		(property "Description" "100nF volume ADC noise filter"
+		(property "Description" "Unpolarized capacitor"
 			(at 0 0 0)
 			(layer "B.Fab")
@@
 			(roundrect_rratio 0.25)
 			(net "GND")
-			(pinfunction "~_1")
 			(pintype "passive")
 		)
@@
 			(roundrect_rratio 0.25)
 			(net "VBUS")
-			(pinfunction "~_2")
 			(pintype "passive")
 		)
@@
 		)
 	)
-	(footprint "microconsole:PCB0029_Footprint"
+	(footprint "microconsole_hardware:PCB0029_Footprint"
 		(layer "B.Cu")
 		(at 153.150001 99.175 180)
@@
 			)
 		)
-		(property "Datasheet" "~"
+		(property "Datasheet" ""
 			(at 0 0 90)
 			(layer "B.Fab")
@@
 			)
 		)
-		(property "Description" "100nF volume ADC noise filter"
+		(property "Description" "Unpolarized capacitor"
 			(at 0 0 90)
 			(layer "B.Fab")
@@
 			(roundrect_rratio 0.212766)
 			(net "GND")
-			(pinfunction "~_1")
 			(pintype "passive")
 		)
@@
 			(roundrect_rratio 0.212766)
 			(net "VBUS")
-			(pinfunction "~_2")
 			(pintype "passive")
 		)

Commit message: Fix TFT library/symbol pin mapping
Updated the TFT symbol and PCB metadata to match the actual LCD pin names and net mapping, corrected the footprint library alias, and removed the stale DRC report generated from the outdated symbol/footprint state.
Connections:
- U1 pad CS: (no net) -> GPIO5 / LCD CS
- U1 pad DC: (no net) -> GPIO9 / LCD DC
- U1 pad GND: (no net) -> GND
- U1 pad LED: (no net) -> VBUS
- U1 pad RESET: (no net) -> GPIO8 / LCD RESET
- U1 pad SCK: (no net) -> GPIO6 / LCD SCK
- U1 pad SD_CS: (no net) -> GPIO13 / SD CS
- U1 pad SD_MISO: (no net) -> GPIO12 / SD MISO
- U1 pad SD_MOSI: (no net) -> GPIO15 / SD MOSI
- U1 pad SD_SCK: (no net) -> GPIO14 / SD SCK
- U1 pad T_CLK: (no net) -> unconnected-(U1-PadT_CLK)_2
- U1 pad T_CS: (no net) -> unconnected-(U1-PadT_CS)_1
- U1 pad T_DIN: (no net) -> unconnected-(U1-PadT_DIN)_1
- U1 pad T_DO: (no net) -> unconnected-(U1-PadT_DO)_1
- U1 pad T_IRQ: (no net) -> unconnected-(U1-PadT_IRQ)
- U1 pad VCC: (no net) -> VBUS
Changed lines of the file:
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@@
 			(unit
 				(name "A")
-				(pins "10" "11" "12" "13" "14" "1" "2" "5" "3" "6" "9" "7" "8" "4")
+				(pins "SD_CS" "SD_MOSI" "SD_MISO" "SD_SCK" "T_CLK" "T_CS" "T_DIN" "T_DO"
+					"T_IRQ" "VCC" "GND" "CS" "RESET" "DC" "MOSI" "SCK" "LED" "MISO"
+				)
 			)
 		)
@@
 			(remove_unused_layers no)
 			(roundrect_rratio 0.15)
+			(net "GPIO5 {slash} LCD CS")
+			(pinfunction "CS_CS")
+			(pintype "input")
 		)
 		(pad "CS" thru_hole roundrect
@@
 			(remove_unused_layers no)
 			(roundrect_rratio 0.15)
+			(net "GPIO5 {slash} LCD CS")
+			(pinfunction "CS_CS")
+			(pintype "input")
 		)
 		(pad "CS" thru_hole roundrect
@@
 			(remove_unused_layers no)
 			(roundrect_rratio 0.15)
+			(net "GPIO5 {slash} LCD CS")
+			(pinfunction "CS_CS")
+			(pintype "input")
 		)
 		(pad "DC" thru_hole roundrect
@@
 			(remove_unused_layers no)
 			(roundrect_rratio 0.15)
+			(net "GPIO9 {slash} LCD DC")
+			(pinfunction "DC_DC")
+			(pintype "input")
 		)
 		(pad "DC" thru_hole roundrect
@@
 			(remove_unused_layers no)
 			(roundrect_rratio 0.15)
+			(net "GPIO9 {slash} LCD DC")
+			(pinfunction "DC_DC")
+			(pintype "input")
 		)
 		(pad "DC" thru_hole roundrect
@@
 			(remove_unused_layers no)
 			(roundrect_rratio 0.15)
+			(net "GPIO9 {slash} LCD DC")
+			(pinfunction "DC_DC")
+			(pintype "input")
 		)
 		(pad "GND" thru_hole roundrect
@@
 			(remove_unused_layers no)
 			(roundrect_rratio 0.15)
+			(net "GND")
+			(pinfunction "GND_GND")
+			(pintype "power_in")
 		)
 		(pad "GND" thru_hole roundrect
@@
 			(remove_unused_layers no)
 			(roundrect_rratio 0.15)
+			(net "GND")
+			(pinfunction "GND_GND")
+			(pintype "power_in")
 		)
 		(pad "GND" thru_hole roundrect
@@
 			(remove_unused_layers no)
 			(roundrect_rratio 0.15)
+			(net "GND")
+			(pinfunction "GND_GND")
+			(pintype "power_in")
 		)
 		(pad "LED" thru_hole roundrect
@@
 			(remove_unused_layers no)
 			(roundrect_rratio 0.15)
+			(net "VBUS")
+			(pinfunction "LED_LED")
+			(pintype "input")
 		)
 		(pad "LED" thru_hole roundrect
@@
 			(remove_unused_layers no)
 			(roundrect_rratio 0.15)
+			(net "VBUS")
+			(pinfunction "LED_LED")
+			(pintype "input")
 		)
 		(pad "LED" thru_hole roundrect
@@
 			(remove_unused_layers no)
 			(roundrect_rratio 0.15)
+			(net "VBUS")
+			(pinfunction "LED_LED")
+			(pintype "input")
 		)
 		(pad "RESET" thru_hole roundrect
@@
 			(remove_unused_layers no)
 			(roundrect_rratio 0.15)
+			(net "GPIO8 {slash} LCD RESET")
+			(pinfunction "RESET_RESET")
+			(pintype "input")
 		)
 		(pad "RESET" thru_hole roundrect
@@
 			(remove_unused_layers no)
 			(roundrect_rratio 0.15)
+			(net "GPIO8 {slash} LCD RESET")
+			(pinfunction "RESET_RESET")
+			(pintype "input")
 		)
 		(pad "RESET" thru_hole roundrect
@@
 			(remove_unused_layers no)
 			(roundrect_rratio 0.15)
+			(net "GPIO8 {slash} LCD RESET")
+			(pinfunction "RESET_RESET")
+			(pintype "input")
 		)
 		(pad "SCK" thru_hole roundrect
@@
 			(remove_unused_layers no)
 			(roundrect_rratio 0.15)
+			(net "GPIO6 {slash} LCD SCK")
+			(pinfunction "SCK_SCK")
+			(pintype "input")
 		)
 		(pad "SCK" thru_hole roundrect
@@
 			(remove_unused_layers no)
 			(roundrect_rratio 0.15)
+			(net "GPIO6 {slash} LCD SCK")
+			(pinfunction "SCK_SCK")
+			(pintype "input")
 		)
 		(pad "SCK" thru_hole roundrect
@@
 			(remove_unused_layers no)
 			(roundrect_rratio 0.15)
+			(net "GPIO6 {slash} LCD SCK")
+			(pinfunction "SCK_SCK")
+			(pintype "input")
 		)
 		(pad "SDI (MOSI)" thru_hole roundrect
@@
 			(remove_unused_layers no)
 			(roundrect_rratio 0.15)
+			(net "GPIO13 {slash} SD CS")
+			(pinfunction "SD_CS_SD_CS")
+			(pintype "input")
 		)
 		(pad "SD_CS" thru_hole roundrect
@@
 			(remove_unused_layers no)
 			(roundrect_rratio 0.15)
+			(net "GPIO13 {slash} SD CS")
+			(pinfunction "SD_CS_SD_CS")
+			(pintype "input")
 		)
 		(pad "SD_CS" thru_hole roundrect
@@
 			(remove_unused_layers no)
 			(roundrect_rratio 0.15)
+			(net "GPIO13 {slash} SD CS")
+			(pinfunction "SD_CS_SD_CS")
+			(pintype "input")
 		)
 		(pad "SD_MISO" thru_hole roundrect
@@
 			(remove_unused_layers no)
 			(roundrect_rratio 0.15)
+			(net "GPIO12 {slash} SD MISO")
+			(pinfunction "SD_MISO_SD_MISO")
+			(pintype "output")
 		)
 		(pad "SD_MISO" thru_hole roundrect
@@
 			(remove_unused_layers no)
 			(roundrect_rratio 0.15)
+			(net "GPIO12 {slash} SD MISO")
+			(pinfunction "SD_MISO_SD_MISO")
+			(pintype "output")
 		)
 		(pad "SD_MISO" thru_hole roundrect
@@
 			(remove_unused_layers no)
 			(roundrect_rratio 0.15)
+			(net "GPIO12 {slash} SD MISO")
+			(pinfunction "SD_MISO_SD_MISO")
+			(pintype "output")
 		)
 		(pad "SD_MOSI" thru_hole roundrect
@@
 			(remove_unused_layers no)
 			(roundrect_rratio 0.15)
+			(net "GPIO15 {slash} SD MOSI")
+			(pinfunction "SD_MOSI_SD_MOSI")
+			(pintype "input")
 		)
 		(pad "SD_MOSI" thru_hole roundrect
@@
 			(remove_unused_layers no)
 			(roundrect_rratio 0.15)
+			(net "GPIO15 {slash} SD MOSI")
+			(pinfunction "SD_MOSI_SD_MOSI")
+			(pintype "input")
 		)
 		(pad "SD_MOSI" thru_hole roundrect
@@
 			(remove_unused_layers no)
 			(roundrect_rratio 0.15)
+			(net "GPIO15 {slash} SD MOSI")
+			(pinfunction "SD_MOSI_SD_MOSI")
+			(pintype "input")
 		)
 		(pad "SD_SCK" thru_hole roundrect
@@
 			(remove_unused_layers no)
 			(roundrect_rratio 0.15)
+			(net "GPIO14 {slash} SD SCK")
+			(pinfunction "SD_SCK_SD_SCK")
+			(pintype "input")
 		)
 		(pad "SD_SCK" thru_hole roundrect
@@
 			(remove_unused_layers no)
 			(roundrect_rratio 0.15)
+			(net "GPIO14 {slash} SD SCK")
+			(pinfunction "SD_SCK_SD_SCK")
+			(pintype "input")
 		)
 		(pad "SD_SCK" thru_hole roundrect
@@
 			(remove_unused_layers no)
 			(roundrect_rratio 0.15)
+			(net "GPIO14 {slash} SD SCK")
+			(pinfunction "SD_SCK_SD_SCK")
+			(pintype "input")
 		)
 		(pad "T_CLK" thru_hole roundrect
@@
 			(remove_unused_layers no)
 			(roundrect_rratio 0.15)
+			(net "unconnected-(U1-PadT_CLK)_1")
+			(pinfunction "T_CLK_T_CLK")
+			(pintype "input+no_connect")
 		)
 		(pad "T_CLK" thru_hole roundrect
@@
 			(remove_unused_layers no)
 			(roundrect_rratio 0.15)
+			(net "unconnected-(U1-PadT_CLK)")
+			(pinfunction "T_CLK_T_CLK")
+			(pintype "input+no_connect")
 		)
 		(pad "T_CLK" thru_hole roundrect
@@
 			(remove_unused_layers no)
 			(roundrect_rratio 0.15)
+			(net "unconnected-(U1-PadT_CLK)_2")
+			(pinfunction "T_CLK_T_CLK")
+			(pintype "input+no_connect")
 		)
 		(pad "T_CS" thru_hole roundrect
@@
 			(remove_unused_layers no)
 			(roundrect_rratio 0.15)
+			(net "unconnected-(U1-PadT_CS)_2")
+			(pinfunction "T_CS_T_CS")
+			(pintype "input+no_connect")
 		)
 		(pad "T_CS" thru_hole roundrect
@@
 			(remove_unused_layers no)
 			(roundrect_rratio 0.15)
+			(net "unconnected-(U1-PadT_CS)")
+			(pinfunction "T_CS_T_CS")
+			(pintype "input+no_connect")
 		)
 		(pad "T_CS" thru_hole roundrect
@@
 			(remove_unused_layers no)
 			(roundrect_rratio 0.15)
+			(net "unconnected-(U1-PadT_CS)_1")
+			(pinfunction "T_CS_T_CS")
+			(pintype "input+no_connect")
 		)
 		(pad "T_DIN" thru_hole roundrect
@@
 			(remove_unused_layers no)
 			(roundrect_rratio 0.15)
+			(net "unconnected-(U1-PadT_DIN)_2")
+			(pinfunction "T_DIN_T_DIN")
+			(pintype "input+no_connect")
 		)
 		(pad "T_DIN" thru_hole roundrect
@@
 			(remove_unused_layers no)
 			(roundrect_rratio 0.15)
+			(net "unconnected-(U1-PadT_DIN)")
+			(pinfunction "T_DIN_T_DIN")
+			(pintype "input+no_connect")
 		)
 		(pad "T_DIN" thru_hole roundrect
@@
 			(remove_unused_layers no)
 			(roundrect_rratio 0.15)
+			(net "unconnected-(U1-PadT_DIN)_1")
+			(pinfunction "T_DIN_T_DIN")
+			(pintype "input+no_connect")
 		)
 		(pad "T_DO" thru_hole roundrect
@@
 			(remove_unused_layers no)
 			(roundrect_rratio 0.15)
+			(net "unconnected-(U1-PadT_DO)_2")
+			(pinfunction "T_DO_T_DO")
+			(pintype "output+no_connect")
 		)
 		(pad "T_DO" thru_hole roundrect
@@
 			(remove_unused_layers no)
 			(roundrect_rratio 0.15)
+			(net "unconnected-(U1-PadT_DO)")
+			(pinfunction "T_DO_T_DO")
+			(pintype "output+no_connect")
 		)
 		(pad "T_DO" thru_hole roundrect
@@
 			(remove_unused_layers no)
 			(roundrect_rratio 0.15)
+			(net "unconnected-(U1-PadT_DO)_1")
+			(pinfunction "T_DO_T_DO")
+			(pintype "output+no_connect")
 		)
 		(pad "T_IRQ" thru_hole roundrect
@@
 			(remove_unused_layers no)
 			(roundrect_rratio 0.15)
+			(net "unconnected-(U1-PadT_IRQ)_2")
+			(pinfunction "T_IRQ_T_IRQ")
+			(pintype "output+no_connect")
 		)
 		(pad "T_IRQ" thru_hole roundrect
@@
 			(remove_unused_layers no)
 			(roundrect_rratio 0.15)
+			(net "unconnected-(U1-PadT_IRQ)_1")
+			(pinfunction "T_IRQ_T_IRQ")
+			(pintype "output+no_connect")
 		)
 		(pad "T_IRQ" thru_hole roundrect
@@
 			(remove_unused_layers no)
 			(roundrect_rratio 0.15)
+			(net "unconnected-(U1-PadT_IRQ)")
+			(pinfunction "T_IRQ_T_IRQ")
+			(pintype "output+no_connect")
 		)
 		(pad "VCC" thru_hole roundrect
@@
 			(remove_unused_layers no)
 			(roundrect_rratio 0.15)
+			(net "VBUS")
+			(pinfunction "VCC_VCC")
+			(pintype "power_in")
 		)
 		(pad "VCC" thru_hole roundrect
@@
 			(remove_unused_layers no)
 			(roundrect_rratio 0.15)
+			(net "VBUS")
+			(pinfunction "VCC_VCC")
+			(pintype "power_in")
 		)
 		(pad "VCC" thru_hole roundrect
@@
 			(remove_unused_layers no)
 			(roundrect_rratio 0.15)
+			(net "VBUS")
+			(pinfunction "VCC_VCC")
+			(pintype "power_in")
 		)
 		(embedded_fonts no)
