File: microconsole_hardware/mc_hw/mc_hw.kicad_pcb (KiCad board)
At the start: 2 copper layers, 200 x 130 mm, 39 parts, among them SW1 DPAD - UP, SW10 START, SW11 L1, SW12 R1, SW13 L2, SW14 R2, SW16 Joystick, SW17 Joystick, SW2 DPAD - DOWN, SW3 DPAD - LEFT, SW4 DPAD - RIGHT, SW5 A, SW6 B, SW7 X, SW8 Y, SW9 SELECT, U1 ILI9341 / ST7796S SPI LCD, U2 MAX98357A, U3 MCP23017x-x-SO

Commit message: hardware update
Parts:
- added D1: LED - GREEN, PCM_SparkFun-Resistor:R_0603_1608Metric, F.Cu at (175.5, 43.0)
- added D2: LED - ORANGE, PCM_SparkFun-Resistor:R_0603_1608Metric, F.Cu at (170.0, 43.0)
- added D3: LED - RED, PCM_SparkFun-Resistor:R_0603_1608Metric, F.Cu at (165.0, 43.0)
- added J2: JST_1mm_4 - BAT IN, PCM_SparkFun-Connector:JST_1x04_P1.0mm_Horizontal_SMD, B.Cu at (194.9, 32.9)
- added J3: JST_1mm_4 - LOAD, PCM_SparkFun-Connector:JST_1x04_P1.0mm_Horizontal_SMD, B.Cu at (186.4, 32.9)
- added JP1: ~, PCM_SparkFun-Jumper:Jumper_2_NO, B.Cu at (187.0, 40.0)
- added JP2: ~, PCM_SparkFun-Jumper:Jumper_2_NO, B.Cu at (193.4, 44.4)
- added R10: 150k, PCM_SparkFun-Resistor:R_0603_1608Metric, B.Cu at (183.9, 49.0)
- added R4: 1k, PCM_SparkFun-Resistor:R_0603_1608Metric, B.Cu at (164.9, 46.5)
- added R5: 1k, PCM_SparkFun-Resistor:R_0603_1608Metric, B.Cu at (169.9, 46.5)
- added R6: 1k, PCM_SparkFun-Resistor:R_0603_1608Metric, B.Cu at (175.4, 46.5)
- added R7: 2k, PCM_SparkFun-Resistor:R_0603_1608Metric, B.Cu at (191.0, 40.0)
- added R8: 1k, PCM_SparkFun-Resistor:R_0603_1608Metric, B.Cu at (183.9, 44.0)
- added R9: 10k, PCM_SparkFun-Resistor:R_0603_1608Metric, B.Cu at (183.9, 46.5)
- added U5: MCP73833_MSOP, PCM_SparkFun-Semiconductor-Standard:MSOP-10_3x3mm_P0.5mm, B.Cu at (188.9, 44.0)
- SW16, SW17: footprint PCM_SparkFun-Switch:Joystick_PTH -> microconsole:Joystick_PTH
- moved C1 36.6 mm to (112.5, 140.0), turned to 0 degrees
- moved R1 26.8 mm to (153.6, 86.9)
- moved R2 26.8 mm to (153.5, 89.5)
- moved C2 15.3 mm to (170.5, 112.0), turned to 90 degrees
- moved LS1 10.0 mm to (150.0, 150.0)
- moved SW17 9.30 mm to (222.5, 129.5)
- moved C9 9.22 mm to (174.0, 112.0), turned to -90 degrees
- moved SW1 7.43 mm to (75.0, 139.5)
- moved SW2 7.43 mm to (75.0, 119.5)
- moved SW3 7.43 mm to (65.0, 129.5)
- moved SW4 7.43 mm to (85.0, 129.5)
Other:
- outline, holes or cut-outs redrawn

Commit message: update
Parts:
- added C16: 1206ZD106KAT2A, project_parts:C1206, F.Cu at (203.4, 147.8)
- added C17: 100nF 50V X7R, project_parts:C_0805_2012Metric_KEMET_IPC-B, F.Cu at (201.8, 129.0)
- added LS2: 8R 1W, Connector_Molex:Molex_PicoBlade_53047-0210_1x02_P1.25mm_Vertical, F.Cu at (218.4, 151.0)
- added LS3: 8R 3W, project_parts:Speaker_WirePads_1x02_P3.50mm_D1.0mm, F.Cu at (242.5, 151.0)
- added R11: RC0805FR-074K7L, project_parts:R0805, F.Cu at (182.4, 146.3)
- added R12: RC0805FR-0710KL, project_parts:R0805, F.Cu at (182.4, 149.3)
- added RV2: 10k Lin, project_parts:Potentiometer_Bourns_PTV09A-2_SideMount_10mm, F.Cu at (178.6, 135.8)
- added SW15: TL3301NF160QG, project_parts:KEY-SMD_4P-L6.0-W6.0-P4.50-LS10.0, F.Cu at (195.8, 125.3)
- added U10: PCM5102APWR, project_parts:TSSOP-20_L6.5-W4.4-P0.65-LS6.4-BL, F.Cu at (196.4, 145.1)
- added U11: S2B-PH-K-S, project_parts:CONN-TH_S2B-PH-K-S-LF-SN, F.Cu at (188.4, 147.7)
- added U6: ADS7828E/2K5, project_parts:TSSOP-16_L5.0-W4.4-P0.65-LS6.4-BL, F.Cu at (203.2, 123.2)
- added U7: MCP23017-E/SO, project_parts:SOIC-28_L18.0-W7.5-P1.27-LS10.3-BL, F.Cu at (182.4, 125.7)
- added U8: PAM8302AADCR, project_parts:SOP-8_L4.9-W3.9-P1.27-LS6.0-BL, F.Cu at (199.8, 136.5)
- added U9: PAM8406DR, project_parts:SOIC-16_L9.9-W3.9-P1.27-LS6.0-BL, F.Cu at (190.8, 136.6)

Commit message: hardware update
Parts:
- removed U1: ILI9341 / ST7796S SPI LCD, microconsole_hardware:TFT
- added DS1: MSP4021, project_parts:LCD_MSP4021_4.0in_SPI_ST7796_1x14_P2.54mm, F.Cu at (94.8, 119.7)
- RV2: footprint project_parts:Potentiometer_Bourns_PTV09A-2_SideMount_10mm -> project_parts:PTV09A2015FB103
