File: microconsole_hardware/mc_hw/mc_hw.kicad_pcb (KiCad board)
At the start: 2 copper layers, 103 parts, among them SW17 Joystick, SW18 Joystick, SW33 TL3301NF160QG, SW34 TL3301NF160QG, SW35 TL3301NF160QG, SW36 TL3301NF160QG, SW37 TL3301NF160QG, SW38 TL3301NF160QG, SW39 TL3301NF160QG, SW40 TL3301NF160QG, SW41 TL3301NF160QG, SW42 TL3301NF160QG, SW43 TL3301NF160QG, SW44 TL3301NF160QG, SW45 TL3301NF160QG, SW46 TL3301NF160QG, U15 ADS7828E/2K5, U16 MCP23017-E/SO, U20 PCM5102APWR, U21 PAM8302AADCR, U22 PAM8406DR, U23 S2B-PH-K-S, U24 S2B-PH-K-S, U6 MCP73833_MSOP

Commit message: small update
Parts:
- moved R45 308.3 mm to (-34.2, 110.0)
- moved R46 308.3 mm to (-39.2, 110.0)
- moved C74 305.7 mm to (-30.9, 105.0)
- moved C75 305.7 mm to (-30.9, 108.0)
- moved C20 200.2 mm to (80.0, 84.1), turned to -90 degrees
- moved R21 187.2 mm to (94.2, 140.0)
- moved C29 176.0 mm to (105.0, 140.0)
- moved C70 155.1 mm to (125.0, 155.0), turned to 0 degrees
- moved C21 153.6 mm to (85.0, 83.4), turned to 90 degrees
- moved C24 152.7 mm to (130.0, 75.0), turned to 90 degrees
- moved C27 151.8 mm to (130.0, 82.5), turned to -90 degrees
- moved C28 145.6 mm to (98.4, 140.0)
- moved R47 136.0 mm to (339.2, 165.0)
- moved R48 136.0 mm to (334.2, 165.0)
- moved R37 135.0 mm to (238.2, 155.0), turned to 0 degrees
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
Commit message: PCB First Pass
Parts:
- removed JP3, JP4: ~, PCM_SparkFun-Jumper:Jumper_2_NO
- removed R19: 10k, PCM_SparkFun-Resistor:R_0603_1608Metric
- removed R20: 150k, PCM_SparkFun-Resistor:R_0603_1608Metric
- removed U24: S2B-PH-K-S, project_parts:CONN-TH_S2B-PH-K-S-LF-SN
- added D1: D_Schottky, PCM_SparkFun-Sensor:Sensirion_DFN-4_1.5x1.5mm_P0.8mm_SHT4x_NoCentralPad, B.Cu at (155.8, 97.8)
- added FB1: FerriteBead_Small, PCM_SparkFun-Capacitor:C_0603_1608Metric, B.Cu at (178.8, 114.5)
- added FB2: FerriteBead_Small, PCM_SparkFun-Capacitor:C_0603_1608Metric, B.Cu at (177.5, 63.0)
- added FB3: FerriteBead_Small, PCM_SparkFun-Capacitor:C_0603_1608Metric, B.Cu at (146.2, 75.8)
- added J2: USB_C_Receptacle_USB2.0_16P, Connector_USB:USB_C_Receptacle_GCT_USB4135-GF-A_6P_TopMnt_Horizontal, B.Cu at (150.0, 60.0)
- added R22: 100k, PCM_SparkFun-Resistor:R_0603_1608Metric, B.Cu at (146.2, 91.8)
- added R49: 5.1k OHM, PCM_SparkFun-Resistor:R_0603_1608Metric, B.Cu at (143.8, 91.0)
- added R50: 5.1k OHM, PCM_SparkFun-Resistor:R_0603_1608Metric, B.Cu at (175.8, 117.5)
- added SW1: SW_Nidec_CAS-120A1, Button_Switch_SMD:Nidec_Copal_CAS-120A, B.Cu at (172.0, 61.0)
- D4, D5, D6, RV4: moved to B.Cu
- R18: value 1k -> 10k
- moved SW41 136.1 mm to (207.2, 62.0), turned to -90 degrees
- moved SW45 136.1 mm to (222.2, 62.0), turned to -90 degrees
- moved SW18 135.8 mm to (222.5, 141.2)
- moved SW40 135.8 mm to (225.0, 105.0)
- moved SW42 135.8 mm to (215.0, 115.0)
- moved SW44 135.8 mm to (215.0, 95.0)
- moved SW46 135.8 mm to (205.0, 105.0)
- moved SW33 135.0 mm to (85.0, 127.0)
- moved SW35 135.0 mm to (85.0, 147.0)
- moved SW37 135.0 mm to (75.0, 137.0)
- moved SW38 135.0 mm to (95.0, 137.0)
- moved SW43 135.0 mm to (77.0, 62.0), turned to 90 degrees
- moved LS9 134.8 mm to (215.0, 78.0), turned to -90 degrees
- moved SW39 134.0 mm to (91.0, 62.0), turned to 90 degrees
- moved R48 132.9 mm to (204.5, 136.0), turned to 90 degrees
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Connections:
- A1 pad 39: unconnected-(A1-VSYS-Pad39)_1 -> VSYS_BAT
- A1 pad 40: VBUS -> VSYS_BAT
- C20 pad 1: VBUS -> VSYS_BAT
- C21 pad 2: VBUS -> VSYS_BAT
- C26 pad 2: VBUS -> VSYS_BAT
- C27 pad 2: VBUS -> VSYS_BAT
- D4 pad 2: VBUS -> USB-VBUS
- D5 pad 2: VBUS -> USB-VBUS
- D6 pad 2: VBUS -> USB-VBUS
- DS2 pad 1: VBUS -> VSYS_BAT
- DS2 pad 8: VBUS -> 3v3
- R12 pad 1: Net-(JP3-A) -> Net-(U6-~{PG})
- R16 pad 1: Net-(U6-~{PG}) -> Net-(U6-STAT1)
- R18 pad 1: Net-(R18-Pad1) -> Net-(U6-THERM)
- R18 pad 2: Net-(U6-THERM) -> GND
- U23 pad 1: VBUS -> BAT+
- U23 pad 2: GND -> Net-(C16-Pad1)
- U6 pad 1: VBUS -> USB-VBUS
- U6 pad 10: VBUS -> BAT+
- U6 pad 2: VBUS -> USB-VBUS
- U6 pad 3: Net-(JP3-A) -> Net-(U6-STAT1)
- U6 pad 9: VBUS -> BAT+
Other:
- board outline added: 161 x 96.5 mm
