File: microconsole_hardware/mc_hw/mc_hw.kicad_pcb (KiCad board)
At the start: 2 copper layers, 161 x 96 mm, 107 parts, among them J2 USB_C_Receptacle_USB2.0_16P, SW1 SW_Nidec_CAS-120A1, SW17 Joystick, SW18 Joystick, SW33 TL3301NF160QG, SW34 TL3301NF160QG, SW35 TL3301NF160QG, SW36 TL3301NF160QG, SW37 TL3301NF160QG, SW38 TL3301NF160QG, SW39 TL3301NF160QG, SW40 TL3301NF160QG, SW41 TL3301NF160QG, SW42 TL3301NF160QG, SW43 TL3301NF160QG, SW44 TL3301NF160QG, SW45 TL3301NF160QG, SW46 TL3301NF160QG, U15 ADS7828E/2K5, U16 MCP23017-E/SO, U20 PCM5102APWR, U21 PAM8302AADCR, U22 PAM8406DR, U23 S2B-PH-K-S, U6 MCP73833_MSOP

Commit message: cleanup2
Parts:
- renumbered C77 to C10, C78 to C11, C79 to C12, C80 to C13, C28 to C4, C29 to C5, C74 to C7, C75 to C8, C76 to C9, D6 to D2, D5 to D3, J2 to J1, R18 to R10, R21 to R11, R45 to R12, R46 to R13, R47 to R14, R48 to R15, R49 to R3, R50 to R4, R22 to R5, R16 to R6, R15 to R7, R12 to R8, R17 to R9, SW37 to SW10, SW44 to SW11, SW43 to SW12, SW38 to SW13, SW46 to SW14, SW45 to SW15, SW17 to SW16, SW18 to SW17, SW33 to SW2, SW40 to SW3, SW39 to SW4, SW34 to SW5, SW35 to SW6, SW42 to SW7, SW41 to SW8, SW36 to SW9, U6 to U1, U23 to U2, U16 to U3, U15 to U4
