File: microconsole_hardware/mc_hw/raw.kicad_sch (KiCad schematic)
At the start: 15 parts, among them SW15 TL3301NF160QG, U10 PCM5102APWR, U11 S2B-PH-K-S, U6 ADS7828E/2K5, U7 MCP23017-E/SO, U8 PAM8302AADCR, U9 PAM8406DR

Commit message: hardware update
Parts:
- removed QD1: QD3508, project_parts:QD3958, symbol project_parts:QD3508
- added DS1: MSP4021, project_parts:LCD_MSP4021_4.0in_SPI_ST7796_1x14_P2.54mm, symbol project_parts:MSP4021
Changed lines of the file:
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@@
-	)
-	(symbol
-		(lib_id "project_parts:QD3508")
-		(at 39.37 43.18 0)
-		(unit 1)
-		(body_style 1)
-		(exclude_from_sim no)
-		(in_bom yes)
-		(on_board yes)
-		(in_pos_files yes)
-		(dnp no)
-		(fields_autoplaced yes)
-		(property "Reference" "QD1"
-			(at 60.96 104.1399 0)
-			(show_name no)
-			(do_not_autoplace no)
-			(effects
-				(font
-					(size 1.27 1.27)
-				)
-				(justify left)
-			)
-		)
-		(property "Value" "QD3508"
-			(at 60.96 106.6799 0)
-			(show_name no)
-			(do_not_autoplace no)
-			(effects
-				(font
-					(size 1.27 1.27)
-				)
-				(justify left)
-			)
-		)
-		(property "Footprint" "project_parts:QD3958"
-			(at 39.37 43.18 0)
-			(hide yes)
-			(show_name no)
-			(do_not_autoplace no)
-			(effects
-				(font
-					(size 1.27 1.27)
-				)
-			)
-		)
-		(property "Datasheet" ""
-			(at 39.37 43.18 0)
-			(hide yes)
-			(show_name no)
-			(do_not_autoplace no)
-			(effects
-				(font
-					(size 1.27 1.27)
-				)
-			)
-		)
-		(property "Description" "4.0 inch SPI TFT display module, 48-pin solder FPC (converted from Altium 4_0inch_SPI.SCHLIB)"
-			(at 39.37 43.18 0)
-			(hide yes)
-			(show_name no)
-			(do_not_autoplace no)
-			(effects
-				(font
-					(size 1.27 1.27)
-				)
-			)
-		)
-		(pin "13"
-		)
-		(pin "25"
-		)
-		(pin "10"
-		)
-		(pin "7"
-		)
-		(pin "14"
-		)
-		(pin "12"
-		)
-		(pin "1"
-		)
-		(pin "3"
-		)
-		(pin "9"
-		)
-		(pin "15"
-		)
-		(pin "19"
-		)
-		(pin "6"
-		)
-		(pin "8"
-		)
-		(pin "21"
-		)
-		(pin "2"
-		)
-		(pin "20"
-		)
-		(pin "18"
-		)
-		(pin "11"
-		)
-		(pin "22"
-		)
-		(pin "16"
-		)
-		(pin "23"
-		)
-		(pin "24"
-		)
-		(pin "4"
-		)
-		(pin "5"
-		)
-		(pin "17"
-		)
-		(pin "26"
-		)
-		(pin "27"
-		)
-		(pin "28"
-		)
-		(pin "29"
-		)
-		(pin "30"
-		)
-		(pin "31"
-		)
-		(pin "32"
-		)
-		(pin "35"
-		)
-		(pin "38"
-		)
-		(pin "47"
-		)
-		(pin "36"
-		)
-		(pin "34"
-		)
-		(pin "40"
-		)
-		(pin "45"
-		)
-		(pin "42"
-		)
-		(pin "37"
-		)
-		(pin "33"
-		)
-		(pin "48"
-		)
-		(pin "44"
-		)
-		(pin "43"
-		)
-		(pin "41"
-		)
-		(pin "39"
-		)
-		(pin "46"
-		)
-		(instances
-			(project "mc_hw"
-				(path "/455a7bd4-49e4-4997-a754-3908b004dd14"
-					(reference "QD1")
-					(unit 1)
-				)
-			)
-		)
 	)
 	(symbol
@@
 					(unit 1)
 				)
+			)
+		)
+	)
+	(symbol
+		(lib_id "project_parts:MSP4021")
+		(at 40.64 99.06 0)
+		(unit 1)
+		(body_style 1)
+		(exclude_from_sim no)
+		(in_bom yes)
+		(on_board yes)
+		(in_pos_files yes)
+		(dnp no)
+		(fields_autoplaced yes)
+		(property "Reference" "DS1"
+			(at 40.9374 74.93 0)
+			(show_name no)
+			(do_not_autoplace no)
+			(effects
+				(font
+					(size 1.27 1.27)
+				)
+			)
+		)
+		(property "Value" "MSP4021"
+			(at 40.9374 77.47 0)
+			(show_name no)
+			(do_not_autoplace no)
+			(effects
+				(font
+					(size 1.27 1.27)
+				)
+			)
+		)
+		(property "Footprint" "project_parts:LCD_MSP4021_4.0in_SPI_ST7796_1x14_P2.54mm"
+			(at 40.64 99.06 0)
+			(hide yes)
+			(show_name no)
+			(do_not_autoplace no)
+			(effects
+				(font
+					(size 1.27 1.27)
+				)
+			)
+		)
+		(property "Datasheet" "https://www.lcdwiki.com/4.0inch_SPI_Module_ST7796"
+			(at 40.64 99.06 0)
+			(hide yes)
+			(show_name no)
+			(do_not_autoplace no)
+			(effects
+				(font
+					(size 1.27 1.27)
+				)
+			)
+		)
+		(property "Description" "4.0in 480x320 SPI TFT module, ST7796S + XPT2046 resistive touch (MSP4020 = no touch), 3.3-5V"
+			(at 40.64 99.06 0)
+			(hide yes)
+			(show_name no)
+			(do_not_autoplace no)
+			(effects
+				(font
+					(size 1.27 1.27)
+				)
+			)
+		)
+		(pin "1"
+		)
+		(pin "3"
+		)
+		(pin "6"
+		)
+		(pin "11"
+		)
+		(pin "7"
+		)
+		(pin "12"
+		)
+		(pin "14"
+		)
+		(pin "4"
+		)
+		(pin "5"
+		)
+		(pin "2"
+		)
+		(pin "10"
+		)
+		(pin "8"
+		)
+		(pin "9"
+		)
+		(pin "13"
+		)
+		(pin "16"
+		)
+		(pin "15"
+		)
+		(pin "18"
+		)
+		(pin "17"
+		)
+		(instances
+			(project "mc_hw"
+				(path "/455a7bd4-49e4-4997-a754-3908b004dd14"
+					(reference "DS1")
+					(unit 1)
+				)
