File: microconsole_hardware/mc_hw/mc_hw.kicad_sch (KiCad schematic)
At the start: 25 parts, among them SW1 DPAD - UP, SW10 START, SW11 L1, SW12 R1, SW13 L2, SW14 R2, SW16 Joystick, SW17 Joystick, SW2 DPAD - DOWN, SW3 DPAD - LEFT, SW4 DPAD - RIGHT, SW5 A, SW6 B, SW7 X, SW8 Y, SW9 SELECT, U1 CR2013-MI2120, U2 MAX98357A, U3 MCP23017x-x-SO

Commit message: quick fix
Parts:
- added C1, C12, C2, C3, C5, C6, C7: 100nF, Capacitor_SMD:C_0603_1608Metric_Pad1.08x0.95mm_HandSolder, symbol Device:C
- added C10, C11, C13, C4, C8, C9: 10uF, Capacitor_SMD:C_0805_2012Metric_Pad1.18x1.45mm_HandSolder, symbol Device:C
- added R3: 10k, PCM_SparkFun-Resistor:R_0603_1608Metric, symbol PCM_SparkFun-Resistor:0.47_0603
- U1: value CR2013-MI2120 -> ILI9341 / ST7796S SPI LCD
Connections:
- net 3v3: now also R1.1, R2.1, U3.9 (V_{DD}), C12.1, C13.2, C2.1, C5.1, C9.2, R3.2
- net AGND: now also C1.1
- net GND: now also U2.17 (PAD), C10.1, C11.1, C12.2, C13.1, C2.2, C3.1, C4.1, C5.2, C6.2, C7.1, C8.1, C9.1
- net GPIO2 / MCP|ADC SDA: now also A1.4 (GPIO2), R1.2; no longer R1.1
- net GPIO28 / VOLUME POT: now also C1.2
- net VBUS: now also U2.4 (~{SD_MODE}), C10.2, C11.2, C3.2, C4.2, C6.1, C7.2, C8.2; no longer U3.9 (V_{DD})
- net GPIO3 / MCP|ADC SCL: now reaches A1.5 (GPIO3), R2.2
- net GPIO3 / MCP|ADC SCL: now also U3.12 (SCL), U4.L3 (SCL)
- net MCP RESET: now reaches U3.18 (~{RESET})
- net MCP RESET: now also R3.1
- removed net GPIO3 / MCP|ADC SCK: R2.1, U3.12 (SCK), U4.L3 (SCL)
- net GPIO4 / ILI MISO renamed GPIO4 / LCD MISO
- net GPIO5 / ILI CS renamed GPIO5 / LCD CS
- net GPIO6 / ILI SCK renamed GPIO6 / LCD SCK
- net GPIO7 / ILI MOSI renamed GPIO7 / LCD MOSI
- net GPIO8 / ILI RESET renamed GPIO8 / LCD RESET
- net GPIO9 / ILI DC renamed GPIO9 / LCD DC
- no-connect marks 24 -> 21
Other:
- moved on the sheet: LS1, R1, R2

Commit message: update symbols and libraries
Connections:
- net 3v3: no longer C5.1
- net MCP GPB3 / L1: now also U3.4 (GPB3)
- net MCP GPB4 / R1: now also U3.5 (GPB4)
- net MCP GPB5 / L2: now also U3.6 (GPB5)
- net MCP GPB6 / R2: now also U3.7 (GPB6)
- net VBUS: now also C5.1
- no-connect marks 21 -> 24
Changed lines of the file:
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@@
 	)
 	(no_connect
+		(at 224.79 25.4)
+	)
+	(no_connect
 		(at 252.73 58.42)
 	)
@@
 	)
 	(no_connect
+		(at 207.01 40.64)
+	)
+	(no_connect
+		(at 207.01 43.18)
+	)
+	(no_connect
 		(at 181.61 143.51)
 	)
@@
 	(wire
 		(pts
+			(xy 78.74 149.86) (xy 81.28 149.86)
+		)
+		(stroke
+			(width 0)
+			(type default)
+		)
+	)
+	(wire
+		(pts
 			(xy 116.84 142.24) (xy 116.84 143.51)
 		)
@@
 	(wire
 		(pts
+			(xy 78.74 147.32) (xy 81.28 147.32)
+		)
+		(stroke
+			(width 0)
+			(type default)
+		)
+	)
+	(wire
+		(pts
 			(xy 219.71 190.5) (xy 217.17 190.5)
 		)
@@
 	(wire
 		(pts
+			(xy 78.74 142.24) (xy 81.28 142.24)
+		)
+		(stroke
+			(width 0)
+			(type default)
+		)
+	)
+	(wire
+		(pts
 			(xy 193.04 219.71) (xy 193.04 222.25)
 		)
@@
 	(wire
 		(pts
+			(xy 78.74 144.78) (xy 81.28 144.78)
+		)
+		(stroke
+			(width 0)
+			(type default)
+		)
+	)
+	(wire
+		(pts
 			(xy 243.84 191.77) (xy 243.84 193.04)
 		)
@@
 		)
 	)
-	(global_label "3v3"
-		(shape input)
-		(at 173.99 149.86 90)
-		(fields_autoplaced yes)
-		(effects
-			(font
-				(size 1.27 1.27)
-			)
-			(justify left)
-		)
-		(property "Intersheetrefs" "${INTERSHEET_REFS}"
-			(at 173.99 143.4882 90)
-			(hide yes)
-			(show_name no)
-			(do_not_autoplace no)
-			(effects
-				(font
-					(size 1.27 1.27)
-				)
-				(justify left)
-			)
-		)
-	)
 	(global_label "MCP GPB2 {slash} START"
 		(shape input)
@@
 		)
 	)
+	(global_label "VBUS"
+		(shape input)
+		(at 173.99 149.86 90)
+		(fields_autoplaced yes)
+		(effects
+			(font
+				(size 1.27 1.27)
+			)
+			(justify left)
+		)
+		(property "Intersheetrefs" "${INTERSHEET_REFS}"
+			(at 173.99 141.9762 90)
+			(hide yes)
+			(show_name no)
+			(do_not_autoplace no)
+			(effects
+				(font
+					(size 1.27 1.27)
+				)
+				(justify left)
+			)
+		)
+	)
 	(global_label "GND"
 		(shape input)
@@
 			)
 		)
-		(property "Description" "100nF volume ADC noise filter"
+		(property "Description" "Unpolarized capacitor"
 			(at 124.46 147.32 0)
 			(hide yes)
@@
 			)
 		)
-		(property "Description" "100nF volume ADC noise filter"
+		(property "Description" "Unpolarized capacitor"
 			(at 274.32 30.48 0)
 			(hide yes)
@@
 			)
 		)
-		(property "Description" "100nF volume ADC noise filter"
+		(property "Description" "Unpolarized capacitor"
 			(at 130.81 185.42 0)
 			(hide yes)
@@
 			)
 		)
-		(property "Description" "100nF volume ADC noise filter"
+		(property "Description" "Unpolarized capacitor"
 			(at 116.84 147.32 0)
 			(hide yes)
@@
 			)
 		)
-		(property "Description" "100nF volume ADC noise filter"
+		(property "Description" "Unpolarized capacitor"
 			(at 124.46 185.42 0)
 			(hide yes)
@@
 			)
 		)
-		(property "Description" "100nF volume ADC noise filter"
+		(property "Description" "Unpolarized capacitor"
 			(at 287.02 30.48 0)
 			(hide yes)
@@
 			)
 		)
-		(property "Description" "100nF volume ADC noise filter"
+		(property "Description" "Unpolarized capacitor"
 			(at 295.91 30.48 0)
 			(hide yes)
@@
 			)
 		)
-		(property "Description" "100nF volume ADC noise filter"
+		(property "Description" "Unpolarized capacitor"
 			(at 173.99 154.94 0)
 			(hide yes)
@@
 			)
 		)
-		(property "Description" "100nF volume ADC noise filter"
+		(property "Description" "Unpolarized capacitor"
 			(at 237.49 187.96 0)
 			(hide yes)
@@
 			)
 		)
-		(property "Description" "100nF volume ADC noise filter"
+		(property "Description" "Unpolarized capacitor"
 			(at 168.91 154.94 0)
 			(hide yes)
@@
 			)
 		)
-		(property "Description" "100nF volume ADC noise filter"
+		(property "Description" "Unpolarized capacitor"
 			(at 243.84 187.96 0)
 			(hide yes)
@@
 			)
 		)
-		(property "Description" "100nF volume ADC noise filter"
+		(property "Description" "Unpolarized capacitor"
 			(at 265.43 30.48 0)
 			(hide yes)
@@
 			)
 		)
-		(property "Description" "100nF volume ADC noise filter"
+		(property "Description" "Unpolarized capacitor"
 			(at 166.37 217.17 0)
 			(hide yes)

Commit message: update hardware
Parts:
- C1, C12, C2, C3, C5, C6, C7: footprint Capacitor_SMD:C_0603_1608Metric_Pad1.08x0.95mm_HandSolder -> (none)
- C10, C11, C13, C4, C8, C9: footprint Capacitor_SMD:C_0805_2012Metric_Pad1.18x1.45mm_HandSolder -> (none)
- LS1: footprint Buzzer_Beeper:Speaker_CUI_CMR-1206S-67 -> (none)
- RV1: footprint Potentiometer_THT:Potentiometer_ACP_CA14-H2,5_Horizontal -> (none)
- SW1, SW10, SW11, SW12, SW13, SW14, SW2, SW3, SW4, SW5, SW6, SW7, SW8, SW9: footprint Button_Switch_SMD:SW_Push_1P1T_NO_E-Switch_TL3301NxxxxxG -> (none)
- U1: footprint Display:CR2013-MI2120 -> microconsole_hardware:TFT; symbol Driver_Display:CR2013-MI2120 -> microconsole:ili9xxx/st7xxxx
- U2: symbol Audio:MAX98357A -> microconsole:MAX98357A
- U4: footprint microconsole:PCB0029_Footprint -> microconsole_hardware:PCB0029_Footprint
Changed lines of the file:
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@@
 	(wire
 		(pts
+			(xy 201.93 209.55) (xy 201.93 208.28)
+		)
+		(stroke
+			(width 0)
+			(type default)
+		)
+	)
+	(wire
+		(pts
 			(xy 204.47 68.58) (xy 207.01 68.58)
 		)
@@
 	(wire
 		(pts
+			(xy 207.01 209.55) (xy 207.01 208.28)
+		)
+		(stroke
+			(width 0)
+			(type default)
+		)
+	)
+	(wire
+		(pts
 			(xy 224.79 138.43) (xy 222.25 138.43)
 		)
@@
 	(global_label "GND"
 		(shape input)
-		(at 207.01 208.28 270)
+		(at 207.01 209.55 270)
 		(fields_autoplaced yes)
 		(effects
@@
 		)
 		(property "Intersheetrefs" "${INTERSHEET_REFS}"
-			(at 207.01 208.28 270)
+			(at 207.01 209.55 270)
 			(hide yes)
 			(show_name no)
@@
 	(global_label "GND"
 		(shape input)
-		(at 201.93 208.28 270)
+		(at 201.93 209.55 270)
 		(fields_autoplaced yes)
 		(effects
@@
 		)
 		(property "Intersheetrefs" "${INTERSHEET_REFS}"
-			(at 201.93 215.1357 90)
+			(at 201.93 216.4057 90)
 			(hide yes)
 			(show_name no)
@@
 			)
 		)
-		(property "Footprint" "Button_Switch_SMD:SW_Push_1P1T_NO_E-Switch_TL3301NxxxxxG"
+		(property "Footprint" ""
 			(at 72.39 67.31 0)
 			(hide yes)
@@
 			)
 		)
-		(property "Footprint" "Button_Switch_SMD:SW_Push_1P1T_NO_E-Switch_TL3301NxxxxxG"
+		(property "Footprint" ""
 			(at 100.33 67.31 0)
 			(hide yes)
@@
 			)
 		)
-		(property "Footprint" "Button_Switch_SMD:SW_Push_1P1T_NO_E-Switch_TL3301NxxxxxG"
+		(property "Footprint" ""
 			(at 52.07 67.31 0)
 			(hide yes)
@@
 			)
 		)
-		(property "Footprint" "Capacitor_SMD:C_0805_2012Metric_Pad1.18x1.45mm_HandSolder"
+		(property "Footprint" ""
 			(at 123.4948 143.51 0)
 			(hide yes)
@@
 			)
 		)
-		(property "Datasheet" "~"
+		(property "Datasheet" ""
 			(at 124.46 147.32 0)
 			(hide yes)
@@
 	)
 	(symbol
+		(lib_name "Joystick_PTH_1")
 		(lib_id "PCM_SparkFun-Switch:Joystick_PTH")
 		(at 50.8 213.36 0)
@@
 			)
 		)
-		(property "Footprint" "Buzzer_Beeper:Speaker_CUI_CMR-1206S-67"
+		(property "Footprint" ""
 			(at 233.68 217.17 0)
 			(hide yes)
@@
 			)
 		)
-		(property "Footprint" "Capacitor_SMD:C_0805_2012Metric_Pad1.18x1.45mm_HandSolder"
+		(property "Footprint" ""
 			(at 273.3548 26.67 0)
 			(hide yes)
@@
 			)
 		)
-		(property "Datasheet" "~"
+		(property "Datasheet" ""
 			(at 274.32 30.48 0)
 			(hide yes)
@@
 			)
 		)
-		(property "Footprint" "Capacitor_SMD:C_0603_1608Metric_Pad1.08x0.95mm_HandSolder"
+		(property "Footprint" ""
 			(at 129.8448 181.61 0)
 			(hide yes)
@@
 			)
 		)
-		(property "Datasheet" "~"
+		(property "Datasheet" ""
 			(at 130.81 185.42 0)
 			(hide yes)
@@
 	)
 	(symbol
-		(lib_name "Joystick_PTH_1")
 		(lib_id "PCM_SparkFun-Switch:Joystick_PTH")
 		(at 111.76 213.36 0)
@@
 			)
 		)
-		(property "Footprint" "Button_Switch_SMD:SW_Push_1P1T_NO_E-Switch_TL3301NxxxxxG"
+		(property "Footprint" ""
 			(at 41.91 22.86 0)
 			(hide yes)
@@
 			)
 		)
-		(property "Footprint" "Capacitor_SMD:C_0603_1608Metric_Pad1.08x0.95mm_HandSolder"
+		(property "Footprint" ""
 			(at 117.8052 151.13 0)
 			(hide yes)
@@
 			)
 		)
-		(property "Datasheet" "~"
+		(property "Datasheet" ""
 			(at 116.84 147.32 0)
 			(hide yes)
@@
 			)
 		)
-		(property "Footprint" "Capacitor_SMD:C_0805_2012Metric_Pad1.18x1.45mm_HandSolder"
+		(property "Footprint" ""
 			(at 123.4948 181.61 0)
 			(hide yes)
@@
 			)
 		)
-		(property "Datasheet" "~"
+		(property "Datasheet" ""
 			(at 124.46 185.42 0)
 			(hide yes)
@@
 			)
 		)
-		(property "Footprint" "Button_Switch_SMD:SW_Push_1P1T_NO_E-Switch_TL3301NxxxxxG"
+		(property "Footprint" ""
 			(at 132.08 22.86 0)
 			(hide yes)
@@
 		(fields_autoplaced yes)
 		(property "Reference" "R1"
-			(at 205.74 26.67 0)
+			(at 201.93 25.3999 90)
 			(show_name no)
 			(do_not_autoplace no)
@@
 					(size 1.27 1.27)
 				)
+				(justify left)
 			)
 		)
 		(property "Value" "4.7k"
-			(at 203.2 26.67 0)
+			(at 201.93 27.9399 90)
 			(show_name no)
 			(do_not_autoplace no)
@@
 					(size 1.27 1.27)
 				)
+				(justify left)
 			)
 		)
@@
 			)
 		)
-		(property "Footprint" "Button_Switch_SMD:SW_Push_1P1T_NO_E-Switch_TL3301NxxxxxG"
+		(property "Footprint" ""
 			(at 69.85 22.86 0)
 			(hide yes)
@@
 			)
 		)
-		(property "Footprint" "Capacitor_SMD:C_0603_1608Metric_Pad1.08x0.95mm_HandSolder"
+		(property "Footprint" ""
 			(at 287.9852 34.29 0)
 			(hide yes)
@@
 			)
 		)
-		(property "Datasheet" "~"
+		(property "Datasheet" ""
 			(at 287.02 30.48 0)
 			(hide yes)
@@
 			)
 		)
-		(property "Footprint" "Button_Switch_SMD:SW_Push_1P1T_NO_E-Switch_TL3301NxxxxxG"
+		(property "Footprint" ""
 			(at 86.36 67.31 0)
 			(hide yes)
@@
 			)
 		)
-		(property "Footprint" "Button_Switch_SMD:SW_Push_1P1T_NO_E-Switch_TL3301NxxxxxG"
+		(property "Footprint" ""
 			(at 55.88 22.86 0)
 			(hide yes)
@@
 			)
 		)
-		(property "Footprint" "Capacitor_SMD:C_0805_2012Metric_Pad1.18x1.45mm_HandSolder"
+		(property "Footprint" ""
 			(at 294.9448 26.67 0)
 			(hide yes)
@@
 			)
 		)
-		(property "Datasheet" "~"
+		(property "Datasheet" ""
 			(at 295.91 30.48 0)
 			(hide yes)
@@
 			)
 		)
-		(property "Footprint" "Button_Switch_SMD:SW_Push_1P1T_NO_E-Switch_TL3301NxxxxxG"
+		(property "Footprint" ""
 			(at 27.94 22.86 0)
 			(hide yes)
@@
 			)
 		)
-		(property "Footprint" "Capacitor_SMD:C_0603_1608Metric_Pad1.08x0.95mm_HandSolder"
+		(property "Footprint" ""
 			(at 174.9552 158.75 0)
 			(hide yes)
@@
 			)
 		)
-		(property "Datasheet" "~"
+		(property "Datasheet" ""
 			(at 173.99 154.94 0)
 			(hide yes)
@@
 	)
 	(symbol
-		(lib_id "Audio:MAX98357A")
+		(lib_id "microconsole:MAX98357A")
 		(at 204.47 195.58 0)
 		(unit 1)
@@
 			)
 		)
-		(property "Footprint" "Button_Switch_SMD:SW_Push_1P1T_NO_E-Switch_TL3301NxxxxxG"
+		(property "Footprint" ""
 			(at 90.17 22.86 0)
 			(hide yes)
@@
 	)
 	(symbol
-		(lib_id "Driver_Display:CR2013-MI2120")
+		(lib_id "microconsole:ili9xxx/st7xxxx")
 		(at 201.93 143.51 0)
 		(unit 1)
@@
 			)
 		)
-		(property "Footprint" "Display:CR2013-MI2120"
-			(at 201.93 161.29 0)
+		(property "Footprint" "microconsole_hardware:TFT"
+			(at 201.93 173.482 0)
 			(hide yes)
 			(show_name no)
@@
 		)
 		(property "Datasheet" "http://pan.baidu.com/s/11Y990"
-			(at 185.42 130.81 0)
+			(at 182.88 127.508 0)
 			(hide yes)
 			(show_name no)
@@
 		)
 		(property "Description" "ILI9341 controller, SPI TFT LCD Display, 9-pin breakout PCB, 4-pin SD card interface, 5V/3.3V"
-			(at 201.93 143.51 0)
+			(at 199.644 170.688 0)
 			(hide yes)
 			(show_name no)
@@
 			)
 		)
-		(property "Footprint" "Potentiometer_THT:Potentiometer_ACP_CA14-H2,5_Horizontal"
-			(at 203.2 241.046 0)
+		(property "Footprint" ""
+			(at 193.04 226.06 0)
+			(hide yes)
 			(show_name no)
 			(do_not_autoplace no)
@@
 			)
 		)
-		(property "Footprint" "Capacitor_SMD:C_0603_1608Metric_Pad1.08x0.95mm_HandSolder"
+		(property "Footprint" ""
 			(at 236.5248 184.15 0)
 			(hide yes)
@@
 			)
 		)
-		(property "Datasheet" "~"
+		(property "Datasheet" ""
 			(at 237.49 187.96 0)
 			(hide yes)
@@
 			)
 		)
-		(property "Footprint" "Button_Switch_SMD:SW_Push_1P1T_NO_E-Switch_TL3301NxxxxxG"
+		(property "Footprint" ""
 			(at 38.1 67.31 0)
 			(hide yes)
@@
 			)
 		)
-		(property "Footprint" "Capacitor_SMD:C_0805_2012Metric_Pad1.18x1.45mm_HandSolder"
+		(property "Footprint" ""
 			(at 167.9448 151.13 0)
 			(hide yes)
@@
 			)
 		)
-		(property "Datasheet" "~"
+		(property "Datasheet" ""
 			(at 168.91 154.94 0)
 			(hide yes)
@@
 		(fields_autoplaced yes)
 		(property "Reference" "U4"
-			(at 91.44 190.5 0)
+			(at 91.44 171.45 0)
 			(show_name no)
 			(do_not_autoplace no)
@@
 			)
 		)
-		(property "Footprint" "microconsole:PCB0029_Footprint"
+		(property "Footprint" "microconsole_hardware:PCB0029_Footprint"
 			(at 91.694 203.2 0)
 			(hide yes)
@@
 			)
 		)
-		(property "Footprint" "Capacitor_SMD:C_0805_2012Metric_Pad1.18x1.45mm_HandSolder"
+		(property "Footprint" ""
 			(at 242.8748 184.15 0)
 			(hide yes)
@@
 			)
 		)
-		(property "Datasheet" "~"
+		(property "Datasheet" ""
 			(at 243.84 187.96 0)
 			(hide yes)
@@
 			)
 		)
-		(property "Footprint" "Capacitor_SMD:C_0603_1608Metric_Pad1.08x0.95mm_HandSolder"
+		(property "Footprint" ""
 			(at 266.3952 34.29 0)
 			(hide yes)
@@
 			)
 		)
-		(property "Datasheet" "~"
+		(property "Datasheet" ""
 			(at 265.43 30.48 0)
 			(hide yes)
@@
 			)
 		)
-		(property "Footprint" "Button_Switch_SMD:SW_Push_1P1T_NO_E-Switch_TL3301NxxxxxG"
+		(property "Footprint" ""
 			(at 114.3 67.31 0)
 			(hide yes)
@@
 			)
 		)
-		(property "Footprint" "Button_Switch_SMD:SW_Push_1P1T_NO_E-Switch_TL3301NxxxxxG"
+		(property "Footprint" ""
 			(at 118.11 22.86 0)
 			(hide yes)
@@
 			)
 		)
-		(property "Footprint" "Capacitor_SMD:C_0603_1608Metric_Pad1.08x0.95mm_HandSolder"
+		(property "Footprint" ""
 			(at 165.4048 213.36 0)
 			(hide yes)
@@
 			)
 		)
-		(property "Datasheet" "~"
+		(property "Datasheet" ""
 			(at 166.37 217.17 0)
 			(hide yes)
@@
 			)
 		)
-		(property "Footprint" "Button_Switch_SMD:SW_Push_1P1T_NO_E-Switch_TL3301NxxxxxG"
+		(property "Footprint" ""
 			(at 104.14 22.86 0)
 			(hide yes)
