File: microconsole_hardware/mc_hw/old.kicad_sch (KiCad schematic)
At the start: 6 parts, among them U2 MAX98357A

Commit message: recover lost pages
Parts:
- removed C1, C3: 100nF, symbol Device:C
- removed C8: 10uF, symbol Device:C
- removed LS1: Speaker, symbol Device:Speaker
- removed RV1: 10k R_Potentiometer, symbol Device:R_Potentiometer
- removed U2: MAX98357A, Package_DFN_QFN:TQFN-16-1EP_3x3mm_P0.5mm_EP1.23x1.23mm, symbol microconsole:MAX98357A
Connections:
- no-connect marks 1 -> 0
