File: microconsole_hardware/mc_hw/old_mc_hw.kicad_sch (KiCad schematic)
At the start: 10 parts

Commit message: recover lost pages
Parts:
- renumbered A2 to A1, C46 to C20, C45 to C21, C50 to C24, C49 to C25, C47 to C26, C48 to C27, DS1 to DS2, R30 to R1, R45 to R2
Changed lines of the file:
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@@
 		(dnp no)
 		(fields_autoplaced yes)
-		(property "Reference" "A2"
+		(property "Reference" "A1"
 			(at 206.6133 151.13 0)
 			(show_name no)
@@
 		)
 		(instances
-			(project "mc_hw"
-				(path "/1b4f24ce-4644-4f48-b948-d506c6ad30e0/522fdc1a-5064-4a45-ac3e-a627e0eb3774"
-					(reference "A2")
-					(unit 1)
-				)
-			)
 			(project "mc_hw"
 				(path "/a5ee2319-7084-42f3-8115-a198bb762e21"
@@
 		(dnp no)
 		(fields_autoplaced yes)
-		(property "Reference" "R30"
+		(property "Reference" "R1"
 			(at 176.53 78.7399 90)
 			(show_name no)
@@
 		)
 		(instances
-			(project "mc_hw"
-				(path "/1b4f24ce-4644-4f48-b948-d506c6ad30e0/522fdc1a-5064-4a45-ac3e-a627e0eb3774"
-					(reference "R30")
-					(unit 1)
-				)
-			)
 			(project "mc_hw"
 				(path "/a5ee2319-7084-42f3-8115-a198bb762e21"
@@
 		(dnp no)
 		(fields_autoplaced yes)
-		(property "Reference" "C50"
+		(property "Reference" "C24"
 			(at 220.98 57.15 90)
 			(show_name no)
@@
 		)
 		(instances
-			(project "mc_hw"
-				(path "/1b4f24ce-4644-4f48-b948-d506c6ad30e0/522fdc1a-5064-4a45-ac3e-a627e0eb3774"
-					(reference "C50")
-					(unit 1)
-				)
-			)
 			(project "mc_hw"
 				(path "/a5ee2319-7084-42f3-8115-a198bb762e21"
@@
 		(in_pos_files yes)
 		(dnp no)
-		(property "Reference" "C46"
+		(property "Reference" "C20"
 			(at 180.086 219.964 0)
 			(show_name no)
@@
 		)
 		(instances
-			(project "mc_hw"
-				(path "/1b4f24ce-4644-4f48-b948-d506c6ad30e0/522fdc1a-5064-4a45-ac3e-a627e0eb3774"
-					(reference "C46")
-					(unit 1)
-				)
-			)
 			(project "mc_hw"
 				(path "/a5ee2319-7084-42f3-8115-a198bb762e21"
@@
 		(in_pos_files yes)
 		(dnp no)
-		(property "Reference" "R45"
+		(property "Reference" "R2"
 			(at 169.672 106.68 0)
 			(show_name no)
@@
 		)
 		(instances
-			(project "mc_hw"
-				(path "/1b4f24ce-4644-4f48-b948-d506c6ad30e0/522fdc1a-5064-4a45-ac3e-a627e0eb3774"
-					(reference "R45")
-					(unit 1)
-				)
-			)
 			(project "mc_hw"
 				(path "/a5ee2319-7084-42f3-8115-a198bb762e21"
@@
 		(dnp no)
 		(fields_autoplaced yes)
-		(property "Reference" "DS1"
+		(property "Reference" "DS2"
 			(at 216.1974 219.71 0)
 			(show_name no)
@@
 		)
 		(instances
-			(project "mc_hw"
-				(path "/1b4f24ce-4644-4f48-b948-d506c6ad30e0/522fdc1a-5064-4a45-ac3e-a627e0eb3774"
-					(reference "DS1")
-					(unit 1)
-				)
-			)
 			(project "mc_hw"
 				(path "/a5ee2319-7084-42f3-8115-a198bb762e21"
@@
 		(dnp no)
 		(fields_autoplaced yes)
-		(property "Reference" "C49"
+		(property "Reference" "C25"
 			(at 220.98 48.26 0)
 			(show_name no)
@@
 		)
 		(instances
-			(project "mc_hw"
-				(path "/1b4f24ce-4644-4f48-b948-d506c6ad30e0/522fdc1a-5064-4a45-ac3e-a627e0eb3774"
-					(reference "C49")
-					(unit 1)
-				)
-			)
 			(project "mc_hw"
 				(path "/a5ee2319-7084-42f3-8115-a198bb762e21"
@@
 		(in_pos_files yes)
 		(dnp no)
-		(property "Reference" "C45"
+		(property "Reference" "C21"
 			(at 166.116 220.98 90)
 			(show_name no)
@@
 		)
 		(instances
-			(project "mc_hw"
-				(path "/1b4f24ce-4644-4f48-b948-d506c6ad30e0/522fdc1a-5064-4a45-ac3e-a627e0eb3774"
-					(reference "C45")
-					(unit 1)
-				)
-			)
 			(project "mc_hw"
 				(path "/a5ee2319-7084-42f3-8115-a198bb762e21"
@@
 		(dnp no)
 		(fields_autoplaced yes)
-		(property "Reference" "C48"
+		(property "Reference" "C27"
 			(at 195.58 57.15 90)
 			(show_name no)
@@
 		)
 		(instances
-			(project "mc_hw"
-				(path "/1b4f24ce-4644-4f48-b948-d506c6ad30e0/522fdc1a-5064-4a45-ac3e-a627e0eb3774"
-					(reference "C48")
-					(unit 1)
-				)
-			)
 			(project "mc_hw"
 				(path "/a5ee2319-7084-42f3-8115-a198bb762e21"
@@
 		(dnp no)
 		(fields_autoplaced yes)
-		(property "Reference" "C47"
+		(property "Reference" "C26"
 			(at 195.58 48.26 0)
 			(show_name no)
@@
 		)
 		(instances
-			(project "mc_hw"
-				(path "/1b4f24ce-4644-4f48-b948-d506c6ad30e0/522fdc1a-5064-4a45-ac3e-a627e0eb3774"
-					(reference "C47")
-					(unit 1)
-				)
-			)
 			(project "mc_hw"
 				(path "/a5ee2319-7084-42f3-8115-a198bb762e21"
@@
 		)
 	)
+	(sheet_instances
+		(path "/"
+			(page "1")
+		)
+	)
+	(embedded_fonts no)
 )
