File: microconsole_hardware/mc_hw/top.kicad_sch (KiCad schematic)
At the start: 0 parts

Commit message: cleanup
Changed lines of the file:
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@@
 	(paper "A4")
 	(sheet
-		(at 95.25 149.86)
-		(size 12.7 20.32)
+		(at 20.32 91.44)
+		(size 68.58 66.04)
 		(exclude_from_sim no)
 		(in_bom yes)
@@
 		)
 		(property "Sheetname" "Audio"
-			(at 95.25 149.1484 0)
+			(at 20.32 90.7284 0)
 			(show_name no)
 			(do_not_autoplace no)
@@
 		)
 		(property "Sheetfile" "audio.kicad_sch"
-			(at 95.25 170.7646 0)
+			(at 20.32 158.0646 0)
 			(show_name no)
 			(do_not_autoplace no)
@@
 	)
 	(sheet
-		(at 119.38 124.46)
-		(size 12.7 20.32)
+		(at 95.25 17.78)
+		(size 68.58 66.04)
 		(exclude_from_sim no)
 		(in_bom yes)
@@
 		)
 		(property "Sheetname" "Battery"
-			(at 119.38 123.7484 0)
+			(at 95.25 17.0684 0)
 			(show_name no)
 			(do_not_autoplace no)
@@
 		)
 		(property "Sheetfile" "battery.kicad_sch"
-			(at 119.38 145.3646 0)
+			(at 95.25 84.4046 0)
 			(show_name no)
 			(do_not_autoplace no)
@@
 	)
 	(sheet
-		(at 95.25 124.46)
-		(size 12.7 20.32)
+		(at 20.32 17.78)
+		(size 68.58 66.04)
 		(exclude_from_sim no)
 		(in_bom yes)
@@
 		)
 		(property "Sheetname" "PicoScreen"
-			(at 95.25 123.7484 0)
+			(at 20.32 17.0684 0)
 			(show_name no)
 			(do_not_autoplace no)
@@
 		)
 		(property "Sheetfile" "mc_hw.kicad_sch"
-			(at 95.25 145.3646 0)
+			(at 20.32 84.4046 0)
 			(show_name no)
 			(do_not_autoplace no)
@@
 	)
 	(sheet
-		(at 119.38 149.86)
-		(size 12.7 20.32)
+		(at 95.25 91.44)
+		(size 68.58 66.04)
 		(exclude_from_sim no)
 		(in_bom yes)
@@
 		)
 		(property "Sheetname" "Buttons"
-			(at 119.38 149.1484 0)
+			(at 95.25 90.7284 0)
 			(show_name no)
 			(do_not_autoplace no)
@@
 		)
 		(property "Sheetfile" "buttons.kicad_sch"
-			(at 119.38 170.7646 0)
+			(at 95.25 158.0646 0)
 			(show_name no)
 			(do_not_autoplace no)
