File: microconsole_hardware/mc_hw/top.kicad_pcb (KiCad board)
At the start: 2 copper layers, 161 x 96 mm, 107 parts, among them J1 USB_C_Receptacle_USB2.0_16P, SW1 SW_Nidec_CAS-120A1, SW10 TL3301NF160QG, SW11 TL3301NF160QG, SW12 TL3301NF160QG, SW13 TL3301NF160QG, SW14 TL3301NF160QG, SW15 TL3301NF160QG, SW16 Joystick, SW17 Joystick, SW2 TL3301NF160QG, SW3 TL3301NF160QG, SW4 TL3301NF160QG, SW5 TL3301NF160QG, SW6 TL3301NF160QG, SW7 TL3301NF160QG, SW8 TL3301NF160QG, SW9 TL3301NF160QG, U1 MCP73833_MSOP, U2 S2B-PH-K-S, U20 PCM5102APWR, U21 PAM8302AADCR, U22 PAM8406DR, U3 MCP23017-E/SO, U4 ADS7828E/2K5

Commit message: fix up everything,
Parts:
- removed A1: RaspberryPi_Pico, Module:RaspberryPi_Pico_Common_Unspecified
- removed the C10 at (182.5, 112.3)
- removed the C13 at (183.3, 114.8)
- removed C20, C24, C53, C58, C61: 100nF 50V X7R, project_parts:C_0805_2012Metric_KEMET_IPC-B
- removed C55: 2.2nF, PCM_SparkFun-Capacitor:C_0805_2012Metric
- removed C59, C60: 0.22uF, PCM_SparkFun-Capacitor:C_0805_2012Metric
- removed C64: 10uF, PCM_SparkFun-Capacitor:C_0805_2012Metric
- removed C66: 1206ZD106KAT2A, project_parts:C1206
- removed C67: 0.47uF, PCM_SparkFun-Capacitor:C_0805_2012Metric
- removed the C7 at (83.7, 111.0)
- removed C71: 1uF, PCM_SparkFun-Capacitor:C_0805_2012Metric
- removed the C9 at (178.8, 112.2)
- removed the FB1 at (178.8, 114.5)
- removed FB3: FerriteBead_Small, PCM_SparkFun-Capacitor:C_0603_1608Metric
- removed R34: 470 OHM, PCM_SparkFun-Resistor:R_0603_1608Metric
- removed R38, R41, R42: 10k OHM, PCM_SparkFun-Resistor:R_0603_1608Metric
- added A2: RaspberryPi_Pico, Module:RaspberryPi_Pico_Common_Unspecified, F.Cu at (114.1, 95.1)
- added C33: 100nF 50V X7R, project_parts:C_0805_2012Metric_KEMET_IPC-B, B.Cu at (145.6, 170.0)
- added C34: 1uF, PCM_SparkFun-Capacitor:C_0805_2012Metric, B.Cu at (159.2, 170.1)
- added C35: 1206ZD106KAT2A, project_parts:C1206, B.Cu at (151.0, 170.1)
- added C36: 100nF 50V X7R, project_parts:C_0805_2012Metric_KEMET_IPC-B, B.Cu at (151.9, 173.3)
- added C37: 1uF, PCM_SparkFun-Capacitor:C_0805_2012Metric, B.Cu at (159.2, 173.4)
- added C38: 10uF, PCM_SparkFun-Capacitor:C_0805_2012Metric, B.Cu at (151.9, 176.3)
- added C39: 1uF, PCM_SparkFun-Capacitor:C_0805_2012Metric, B.Cu at (159.2, 176.8)
- added C40: 100nF 50V X7R, project_parts:C_0805_2012Metric_KEMET_IPC-B, B.Cu at (160.1, 179.9)
- added C41: 1206ZD106KAT2A, project_parts:C1206, B.Cu at (160.1, 183.0)
- added C42: 0.47uF, PCM_SparkFun-Capacitor:C_0805_2012Metric, B.Cu at (160.1, 186.1)
- added C43: 1uF, PCM_SparkFun-Capacitor:C_0805_2012Metric, B.Cu at (125.3, 173.7)
- added C44: 100nF 50V X7R, project_parts:C_0805_2012Metric_KEMET_IPC-B, B.Cu at (125.3, 170.6)
- added C45: 1206ZD106KAT2A, project_parts:C1206, B.Cu at (88.5, 83.0)
- added C46: 100nF 50V X7R, project_parts:C_0805_2012Metric_KEMET_IPC-B, B.Cu at (91.0, 83.0)
- added C47: 1206ZD106KAT2A, project_parts:C1206, B.Cu at (136.7, 174.1)
- added C48: 100nF 50V X7R, project_parts:C_0805_2012Metric_KEMET_IPC-B, B.Cu at (137.6, 183.7)
- added C49: 1206ZD106KAT2A, project_parts:C1206, B.Cu at (136.7, 177.4)
- added C50: 100nF 50V X7R, project_parts:C_0805_2012Metric_KEMET_IPC-B, B.Cu at (137.6, 186.7)
- added FB4: FerriteBead_Small, PCM_SparkFun-Capacitor:C_0603_1608Metric, B.Cu at (129.6, 170.3)
- added FB5: FerriteBead_Small, PCM_SparkFun-Capacitor:C_0603_1608Metric, B.Cu at (129.6, 172.9)
- added Q1: Q_PMOS_GSD, Package_TO_SOT_THT:TO-92, F.Cu at (186.1, 63.4)
- added R28: 2.2k OHM, PCM_SparkFun-Resistor:R_0603_1608Metric, B.Cu at (160.4, 188.8)
- added R29: 22k OHM, PCM_SparkFun-Resistor:R_0603_1608Metric, B.Cu at (160.4, 191.3)
- added R30: 4.7k, PCM_SparkFun-Resistor:R_0603_1608Metric, B.Cu at (137.8, 189.5)
- added R45: 4.7k, PCM_SparkFun-Resistor:R_0603_1608Metric, B.Cu at (137.8, 192.0)
- C1: renamed from C65; value 1uF -> 10uF
- C11: renamed from C26; value 1206ZD106KAT2A -> 100nF 50V X7R; footprint project_parts:C1206 -> project_parts:C_0805_2012Metric_KEMET_IPC-B
- C14: renamed from C68; value 1uF -> 100nF 50V X7R; footprint PCM_SparkFun-Capacitor:C_0805_2012Metric -> project_parts:C_0805_2012Metric_KEMET_IPC-B
- C15: renamed from C72; value 0.47uF -> 1206ZD106KAT2A; footprint PCM_SparkFun-Capacitor:C_0805_2012Metric -> project_parts:C1206
- C16: renamed from C54; value 1206ZD106KAT2A -> 100nF 50V X7R; footprint project_parts:C1206 -> project_parts:C_0805_2012Metric_KEMET_IPC-B
- C18: renamed from C52; value 1206ZD106KAT2A -> 2.2nF; footprint project_parts:C1206 -> PCM_SparkFun-Capacitor:C_0805_2012Metric
- C19: renamed from C69; value 1206ZD106KAT2A -> 2.2nF; footprint project_parts:C1206 -> PCM_SparkFun-Capacitor:C_0805_2012Metric
- C2: renamed from C25; value 1206ZD106KAT2A -> 10uF
- C22: renamed from C57; value 33nF -> 2.2uF
- C23: renamed from C8; value 100nF 50V X7R -> 33nF; footprint project_parts:C_0805_2012Metric_KEMET_IPC-B -> PCM_SparkFun-Capacitor:C_0805_2012Metric
- C28: renamed from C5; value 100nF 50V X7R -> 2.2uF; footprint project_parts:C_0805_2012Metric_KEMET_IPC-B -> PCM_SparkFun-Capacitor:C_0805_2012Metric
- C30: renamed from C70; value 100nF 50V X7R -> 0.22uF; footprint project_parts:C_0805_2012Metric_KEMET_IPC-B -> PCM_SparkFun-Capacitor:C_0805_2012Metric
- C31: renamed from C12; value 100nF 50V X7R -> 0.22uF; footprint project_parts:C_0805_2012Metric_KEMET_IPC-B -> PCM_SparkFun-Capacitor:C_0805_2012Metric
- C32: renamed from C11; value 100nF 50V X7R -> 0.47uF; footprint project_parts:C_0805_2012Metric_KEMET_IPC-B -> PCM_SparkFun-Capacitor:C_0805_2012Metric
- C4: renamed from C3; value 2.2uF -> 1206ZD106KAT2A; footprint PCM_SparkFun-Capacitor:C_0805_2012Metric -> project_parts:C1206
- C5: renamed from C6; value 2.2uF -> 100nF 50V X7R; footprint PCM_SparkFun-Capacitor:C_0805_2012Metric -> project_parts:C_0805_2012Metric_KEMET_IPC-B
- C7: renamed from C73; value 1uF -> 100nF 50V X7R; footprint PCM_SparkFun-Capacitor:C_0805_2012Metric -> project_parts:C_0805_2012Metric_KEMET_IPC-B
- C8: renamed from C56; value 2.2nF -> 100nF 50V X7R; footprint PCM_SparkFun-Capacitor:C_0805_2012Metric -> project_parts:C_0805_2012Metric_KEMET_IPC-B
- C9: renamed from C62; value 100nF 50V X7R -> 1uF; footprint project_parts:C_0805_2012Metric_KEMET_IPC-B -> PCM_SparkFun-Capacitor:C_0805_2012Metric
- D1: renamed from D4; value LED - ORANGE -> D_Schottky; footprint PCM_SparkFun-Resistor:R_0603_1608Metric -> PCM_SparkFun-Sensor:Sensirion_DFN-4_1.5x1.5mm_P0.8mm_SHT4x_NoCentralPad
- D2: renamed from D3; value LED - GREEN -> LED - RED; moved to F.Cu
- D3: renamed from D2; value LED - RED -> LED - GREEN; moved to F.Cu
- D4: renamed from D1; value D_Schottky -> LED - ORANGE; footprint PCM_SparkFun-Sensor:Sensirion_DFN-4_1.5x1.5mm_P0.8mm_SHT4x_NoCentralPad -> PCM_SparkFun-Resistor:R_0603_1608Metric; moved to F.Cu
- LS2: renamed from LS9; value 8R 1W -> 8R 3W; footprint Connector_Molex:Molex_PicoBlade_53047-0210_1x02_P1.25mm_Vertical -> project_parts:Speaker_WirePads_1x02_P3.50mm_D1.0mm
- LS3: renamed from LS7; value 8R 3W -> 8R 1W; footprint project_parts:Speaker_WirePads_1x02_P3.50mm_D1.0mm -> Connector_Molex:Molex_PicoBlade_53047-0210_1x02_P1.25mm_Vertical
- R10: renamed from R40; value 2.2k OHM -> 10k
- R11: renamed from R5; value 100k -> 10k
- R12: renamed from R8; value 1k -> 1k OHM
- R13: renamed from R10; value 10k -> 1k OHM
- R14: renamed from R7; value 1k -> 1k OHM
- R15: renamed from R6; value 1k -> 1k OHM
- R16: renamed from R9; value 2k -> 10k OHM
- R17: renamed from R37; value 100k OHM -> 10k OHM
- R18: renamed from R39; value 22k OHM -> 470 OHM
- R19: renamed from R36; value 4.7k OHM -> 470 OHM
- R21: renamed from R31; value 10k OHM -> 4.7k OHM
- R22: renamed from R13; value 1k OHM -> 22k OHM
- R23: renamed from R12; value 1k OHM -> 2.2k OHM
- R24: renamed from R11; value 10k -> 100k OHM
- R25: renamed from R4; value 5.1k OHM -> 10k OHM
- R26: renamed from R15; value 1k OHM -> 10k OHM
- R27: renamed from R14; value 1k OHM -> 10k OHM
- R3: renamed from R33; value 470 OHM -> 5.1k OHM
- R4: renamed from R44; value 22k OHM -> 5.1k OHM
- R5: renamed from R43; value 2.2k OHM -> 100k
- R6: renamed from R32; value 10k OHM -> 1k
- R7: renamed from R2; value 4.7k -> 1k
- R8: renamed from R1; value 4.7k -> 1k
- R9: renamed from R3; value 5.1k OHM -> 2k
- SW1: renamed from SW15; value TL3301NF160QG -> SW_Nidec_CAS-120A1; footprint project_parts:KEY-SMD_4P-L6.0-W6.0-P4.50-LS10.0 -> Button_Switch_SMD:Nidec_Copal_CAS-120A
- SW16: renamed from SW1; value SW_Nidec_CAS-120A1 -> Joystick; footprint Button_Switch_SMD:Nidec_Copal_CAS-120A -> project_parts:GINFULL HallEffect Joystick PTH; moved to F.Cu
- SW17: renamed from SW14; value TL3301NF160QG -> Joystick; footprint project_parts:KEY-SMD_4P-L6.0-W6.0-P4.50-LS10.0 -> project_parts:GINFULL HallEffect Joystick PTH
- SW3: renamed from SW17; value Joystick -> TL3301NF160QG; footprint project_parts:GINFULL HallEffect Joystick PTH -> project_parts:KEY-SMD_4P-L6.0-W6.0-P4.50-LS10.0
- SW4: renamed from SW16; value Joystick -> TL3301NF160QG; footprint project_parts:GINFULL HallEffect Joystick PTH -> project_parts:KEY-SMD_4P-L6.0-W6.0-P4.50-LS10.0
- U1: renamed from U22; value PAM8406DR -> MCP73833_MSOP; footprint project_parts:SOIC-16_L9.9-W3.9-P1.27-LS6.0-BL -> PCM_SparkFun-Semiconductor-Standard:MSOP-10_3x3mm_P0.5mm
- U2: renamed from U20; value PCM5102APWR -> S2B-PH-K-S; footprint project_parts:TSSOP-20_L6.5-W4.4-P0.65-LS6.4-BL -> project_parts:CONN-TH_S2B-PH-K-S-LF-SN
- U3: renamed from U21; value PAM8302AADCR -> MCP23017-E/SO; footprint project_parts:SOP-8_L4.9-W3.9-P1.27-LS6.0-BL -> project_parts:SOIC-28_L18.0-W7.5-P1.27-LS10.3-BL
- U4: renamed from U1; value MCP73833_MSOP -> ADS7828E/2K5; footprint PCM_SparkFun-Semiconductor-Standard:MSOP-10_3x3mm_P0.5mm -> project_parts:TSSOP-16_L5.0-W4.4-P0.65-LS6.4-BL
- U5: renamed from U2; value S2B-PH-K-S -> PCM5102APWR; footprint project_parts:CONN-TH_S2B-PH-K-S-LF-SN -> project_parts:TSSOP-20_L6.5-W4.4-P0.65-LS6.4-BL
- U6: renamed from U3; value MCP23017-E/SO -> PAM8302AADCR; footprint project_parts:SOIC-28_L18.0-W7.5-P1.27-LS10.3-BL -> project_parts:SOP-8_L4.9-W3.9-P1.27-LS6.0-BL
- U7: renamed from U4; value ADS7828E/2K5 -> PAM8406DR; footprint project_parts:TSSOP-16_L5.0-W4.4-P0.65-LS6.4-BL -> project_parts:SOIC-16_L9.9-W3.9-P1.27-LS6.0-BL
- moved R27 226.8 mm to (74.5, -36.0)
- moved C32 226.5 mm to (77.0, -36.0)
- moved R26 226.5 mm to (70.0, -43.0)
- moved C31 225.7 mm to (70.0, -40.0), turned to 180 degrees
- moved C23 141.7 mm to (69.2, -35.5)
- moved R22 141.7 mm to (67.2, -37.5)
- moved R23 141.7 mm to (72.3, -30.5)
- moved SW11 129.4 mm to (215.0, 92.0)
- moved SW5 125.9 mm to (173.0, 136.5)
- moved R11 119.7 mm to (206.0, -12.0)
- moved SW17 119.7 mm to (86.3, 105.0)
- moved C4 118.5 mm to (226.0, -14.5)
- moved U3 117.9 mm to (214.2, -16.6)
- moved C5 114.7 mm to (223.5, -14.5), turned to -90 degrees
- moved C7 104.5 mm to (80.0, 102.6), turned to -90 degrees
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- renumbered C51 to C10, C27 to C12, C21 to C13, C63 to C17, C4 to C29, DS2 to DS1, FB2 to FB1, LS8 to LS1, R35 to R20, RV4 to RV1, SW6 to SW10, SW4 to SW11, SW2 to SW12, SW5 to SW13, SW11 to SW14, SW7 to SW15, SW13 to SW2, SW12 to SW5, SW10 to SW6, SW9 to SW7, SW3 to SW9
Connections:
- C1 pad 1: AMP_VDD -> GND
- C1 pad 2: GND -> USB-VBUS
- C10 pad 1: GND -> 3v3
- C10 pad 2: 3v3_AUDIO -> GND
- C11 pad 2: VSYS_BAT -> FILTERED - IO2 / Right Stick X
- C12 pad 2: VSYS_BAT -> FILTERED - IO3 / Right Stick Y
- C13 pad 2: VSYS_BAT -> 3v3
- C14 pad 2: AMP_VDD -> 3v3_AUDIO
- C15 pad 1: Net-(U22-INR) -> GND
- C15 pad 2: Net-(C72-Pad2) -> GND
- C16 pad 2: GND -> 3v3_AUDIO
- C18 pad 1: GND -> DAC_L
- C19 pad 1: AMP_VDD -> DAC_R
- C2 pad 1: 3v3 -> Net-(C2-Pad1)
- C22 pad 1: CENTER_FEED -> Net-(U5-VNEG)
- C23 pad 1: GND -> CENTER_FEED
- C23 pad 2: FILTERED - IO1 / Left Stick Y -> GND
- C28 pad 1: 3v3 -> Net-(U5-CAPP)
- C28 pad 2: GND -> Net-(U5-CAPM)
- C29 pad 2: 3v3 -> AMP_VDD
- C30 pad 1: GND -> CENTER_FEED
- C30 pad 2: VOL_ADC -> Net-(U6-IN+)
- C31 pad 1: GND -> Net-(U6-IN-)
- C31 pad 2: FILTERED - IO3 / Right Stick Y -> GND
- C32 pad 1: GND -> Net-(U7-INL)
- C32 pad 2: FILTERED - IO2 / Right Stick X -> Net-(C32-Pad2)
- C4 pad 1: Net-(U20-CAPP) -> GND
- C4 pad 2: Net-(U20-CAPM) -> 3v3
- C5 pad 1: Net-(U20-VNEG) -> 3v3
- C7 pad 2: AMP_VDD -> FILTERED - IO0 / Left Stick X
- C8 pad 1: DAC_R -> GND
- C8 pad 2: GND -> FILTERED - IO1 / Left Stick Y
- C9 pad 1: GND -> 3v3_ADC
- C9 pad 2: 3v3_AUDIO -> GND
- D1 pad 1: Net-(D4-K) -> SYS_RAW
- D2 pad 1: Net-(D3-K) -> Net-(D2-K)
- D3 pad 1: Net-(D2-K) -> Net-(D3-K)
- D4 pad 1: SYS_RAW -> Net-(D4-K)
- FB1 pad 1: VSYS_BAT -> 3v3
- FB1 pad 2: AMP_VDD -> 3v3_ADC
- LS1 pad 1: Net-(LS8-+_(red)) -> Net-(LS1-+_(red))
- LS1 pad 2: Net-(LS8--_(black)) -> Net-(LS1--_(black))
- LS2 pad 1: Net-(LS9-+_(red)) -> Net-(LS2-+)
- LS2 pad 2: Net-(LS9--_(black)) -> Net-(LS2--)
- LS3 pad 1: Net-(LS7-+) -> Net-(LS3-+_(red))
- LS3 pad 2: Net-(LS7--) -> Net-(LS3--_(black))
- R10 pad 1: Net-(C67-Pad2) -> Net-(U1-THERM)
- R11 pad 1: USB-VBUS -> MCP RESET
- R11 pad 2: GND -> 3v3
- R12 pad 1: Net-(U1-~{PG}) -> FILTERED - IO0 / Left Stick X
- R12 pad 2: Net-(D4-K) -> IO0 / Left Stick X
- R13 pad 1: Net-(U1-THERM) -> FILTERED - IO1 / Left Stick Y
- R13 pad 2: GND -> IO1 / Left Stick Y
- R14 pad 1: Net-(U1-STAT2) -> FILTERED - IO2 / Right Stick X
- R14 pad 2: Net-(D3-K) -> IO2 / Right Stick X
- R15 pad 1: Net-(U1-STAT1) -> FILTERED - IO3 / Right Stick Y
- R15 pad 2: Net-(D2-K) -> IO3 / Right Stick Y
- R16 pad 1: Net-(U1-PROG) -> CENTER_MIX
- R16 pad 2: GND -> DAC_L
- R17 pad 1: AMP_VDD -> DAC_R
- R17 pad 2: Net-(U21-~{SD}) -> CENTER_MIX
- R18 pad 1: Net-(C67-Pad2) -> Net-(U5-OUTL)
- R19 pad 1: CENTER_FEED -> Net-(U5-OUTR)
- R19 pad 2: GND -> DAC_R
- R21 pad 1: CENTER_MIX -> CENTER_FEED
- R21 pad 2: DAC_L -> GND
- R22 pad 1: FILTERED - IO1 / Left Stick Y -> Net-(C32-Pad2)
- R22 pad 2: IO1 / Left Stick Y -> DAC_L
- R23 pad 1: FILTERED - IO0 / Left Stick X -> Net-(C32-Pad2)
- R23 pad 2: IO0 / Left Stick X -> GND
- R24 pad 1: MCP RESET -> AMP_VDD
- R24 pad 2: 3v3 -> Net-(U6-~{SD})
- R25 pad 1: GND -> Net-(U7-~{MUTE})
- R25 pad 2: Net-(J1-CC2) -> AMP_VDD
- R26 pad 1: FILTERED - IO3 / Right Stick Y -> 3v3_AUDIO
- R26 pad 2: IO3 / Right Stick Y -> Net-(U5-XSMT)
- R27 pad 1: FILTERED - IO2 / Right Stick X -> AMP_VDD
- R27 pad 2: IO2 / Right Stick X -> Net-(U7-~{SHDN})
- R3 pad 1: Net-(U20-OUTL) -> Net-(J1-CC1)
- R3 pad 2: DAC_L -> GND
- R4 pad 1: Net-(C72-Pad2) -> GND
- R4 pad 2: DAC_R -> Net-(J1-CC2)
- R5 pad 1: Net-(C72-Pad2) -> USB-VBUS
- R6 pad 1: DAC_R -> Net-(U1-STAT1)
- R6 pad 2: CENTER_MIX -> Net-(D2-K)
- R7 pad 1: 3v3 -> Net-(U1-STAT2)
- R7 pad 2: GPIO3 / MCP|ADC SCL -> Net-(D3-K)
- R8 pad 1: 3v3 -> Net-(U1-~{PG})
- R8 pad 2: GPIO2 / MCP|ADC SDA -> Net-(D4-K)
- R9 pad 1: Net-(J1-CC1) -> Net-(U1-PROG)
- SW1 pad 1: GND -> VSYS_BAT
- SW1 pad 2: unconnected-(SW15-Pad2) (its old number) -> SYS_RAW
- SW10 pad 4: MCP GPA1 / DPAD - DOWN -> MCP GPA2 / DPAD - LEFT
- SW11 pad 4: MCP GPB3 / L1 -> MCP GPA6 / X
- SW12 pad 4: MCP GPA0 / DPAD - UP -> MCP GPB5 / L2
- SW13 pad 4: MCP GPB1 / SELECT -> MCP GPA3 / DPAD - RIGHT
- SW14 pad 4: MCP GPA6 / X -> MCP GPB0 / Y
- SW15 pad 4: MCP GPA5 / B -> MCP GPB6 / R2
- SW2 pad 4: MCP GPA3 / DPAD - RIGHT -> MCP GPA0 / DPAD - UP
- SW5 pad 4: MCP GPB5 / L2 -> MCP GPB1 / SELECT
- SW6 pad 4: MCP GPA2 / DPAD - LEFT -> MCP GPA1 / DPAD - DOWN
- SW7 pad 4: MCP GPB2 / START -> MCP GPA5 / B
- SW9 pad 4: MCP GPA4 / A -> MCP GPB2 / START
- U1 pad 1: Net-(LS8-+_(red)) -> USB-VBUS
- U1 pad 10: Net-(U22-INR) -> BAT+
- U1 pad 2: GND -> USB-VBUS
- U1 pad 3: Net-(LS8--_(black)) -> Net-(U1-STAT1)
- U1 pad 4: AMP_VDD -> Net-(U1-STAT2)
- U1 pad 5: Net-(U22-~{MUTE}) -> GND
- U1 pad 6: AMP_VDD -> Net-(U1-PROG)
- U1 pad 7: Net-(U22-INL) -> Net-(U1-~{PG})
- U1 pad 8: Net-(U22-VREF) -> Net-(U1-THERM)
- U1 pad 9: AMP_VDD -> BAT+
- U2 pad 1: 3v3_AUDIO -> BAT+
- U2 pad 2: Net-(U20-CAPP) -> Net-(C2-Pad1)
- U3 pad 1: Net-(U21-~{SD}) -> MCP GPB0 / Y
- U3 pad 2: unconnected-(U21-NC-Pad2) -> MCP GPB1 / SELECT
- U3 pad 3: Net-(U21-IN+) -> MCP GPB2 / START
- U3 pad 4: Net-(U21-IN-) -> MCP GPB3 / L1
- U3 pad 5: Net-(LS7--) -> MCP GPB4 / R1
- U3 pad 6: AMP_VDD -> MCP GPB5 / L2
- U3 pad 7: GND -> MCP GPB6 / R2
- U3 pad 8: Net-(LS7-+) -> unconnected-(U3-GPB7-Pad8)
- U4 pad 1: USB-VBUS -> FILTERED - IO0 / Left Stick X
- U4 pad 10: BAT+ -> 3v3_ADC
- U4 pad 2: USB-VBUS -> FILTERED - IO1 / Left Stick Y
- U4 pad 3: Net-(U1-STAT1) -> FILTERED - IO2 / Right Stick X
- U4 pad 4: Net-(U1-STAT2) -> FILTERED - IO3 / Right Stick Y
- U4 pad 5: GND -> VOL_ADC
- U4 pad 6: Net-(U1-PROG) -> unconnected-(U4-CH5-Pad6)
- U4 pad 7: Net-(U1-~{PG}) -> unconnected-(U4-CH6-Pad7)
- U4 pad 8: Net-(U1-THERM) -> unconnected-(U4-CH7-Pad8)
- U4 pad 9: BAT+ -> GND
- U5 pad 1: BAT+ -> 3v3_AUDIO
- U5 pad 2: Net-(C2-Pad1) -> Net-(U5-CAPP)
- U6 pad 1: MCP GPB0 / Y -> Net-(U6-~{SD})
- U6 pad 2: MCP GPB1 / SELECT -> unconnected-(U6-NC-Pad2)
- U6 pad 3: MCP GPB2 / START -> Net-(U6-IN+)
- U6 pad 4: MCP GPB3 / L1 -> Net-(U6-IN-)
- U6 pad 5: MCP GPB4 / R1 -> Net-(LS2--)
- U6 pad 6: MCP GPB5 / L2 -> AMP_VDD
- U6 pad 7: MCP GPB6 / R2 -> GND
- U6 pad 8: unconnected-(U3-GPB7-Pad8) -> Net-(LS2-+)
- U7 pad 1: FILTERED - IO0 / Left Stick X -> Net-(LS1-+_(red))
- U7 pad 10: 3v3_ADC -> Net-(U7-INR)
- U7 pad 12: GND -> Net-(U7-~{SHDN})
- U7 pad 13: GND -> AMP_VDD
- U7 pad 14: GPIO3 / MCP|ADC SCL -> Net-(LS3--_(black))
- U7 pad 15: GPIO2 / MCP|ADC SDA -> GND
- U7 pad 16: 3v3 -> Net-(LS3-+_(red))
- U7 pad 2: FILTERED - IO1 / Left Stick Y -> GND
- U7 pad 3: FILTERED - IO2 / Right Stick X -> Net-(LS1--_(black))
- U7 pad 4: FILTERED - IO3 / Right Stick Y -> AMP_VDD
- U7 pad 5: VOL_ADC -> Net-(U7-~{MUTE})
- U7 pad 6: unconnected-(U4-CH5-Pad6) -> AMP_VDD
- U7 pad 7: unconnected-(U4-CH6-Pad7) -> Net-(U7-INL)
- U7 pad 8: unconnected-(U4-CH7-Pad8) -> Net-(U7-VREF)
- U7 pad 9: GND -> AMP_VDD

Commit message: prototype pass 1
Parts:
- A2: moved to B.Cu
- C14, C16, C36, C40: value 100nF 50V X7R -> 100nF
- moved C31 188.9 mm to (168.9, 121.0), turned to 0 degrees
- moved C23 187.0 mm to (173.9, 119.5), turned to -90 degrees
- moved R22 175.5 mm to (173.4, 102.1), turned to 180 degrees
- moved C32 172.0 mm to (178.2, 103.1)
- moved R23 169.1 mm to (175.9, 103.1), turned to -90 degrees
- moved R27 161.0 mm to (170.7, 93.1)
- moved C4 158.8 mm to (196.8, 141.6)
- moved C5 158.8 mm to (194.2, 141.6)
- moved R11 158.8 mm to (176.8, 144.1)
- moved U3 158.8 mm to (185.0, 139.5)
- moved R26 157.4 mm to (142.2, 96.8), turned to 0 degrees
- moved C10 117.2 mm to (121.0, 133.5), turned to 0 degrees
- moved R30 117.1 mm to (100.5, 78.5), turned to 0 degrees
- moved R45 117.1 mm to (100.5, 81.0), turned to 0 degrees
- moved C13 117.1 mm to (121.5, 131.0), turned to 180 degrees
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
Commit message: cleanup
Parts:
- C14, C16, C36, C40: value 100nF -> 100nF 50V X7R
Changed lines of the file:
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@@
 	)
 	(footprint "Button_Switch_SMD:Nidec_Copal_CAS-120A"
+		(locked yes)
 		(layer "F.Cu")
 		(at 132 60.5 -90)
@@
 				(font
 					(size 1.27 1.27)
+					(thickness 0.15)
 				)
 			)
@@
 				(font
 					(size 1.27 1.27)
+					(thickness 0.15)
 				)
 			)
@@
 				(font
 					(size 1.27 1.27)
+					(thickness 0.15)
 				)
 			)
@@
 				(font
 					(size 1.27 1.27)
+					(thickness 0.15)
 				)
 			)
@@
 				(font
 					(size 1.27 1.27)
+					(thickness 0.15)
 				)
 				(justify mirror)
@@
 				(font
 					(size 1.27 1.27)
+					(thickness 0.15)
 				)
 				(justify mirror)
@@
 			)
 		)
-		(property "Value" "100nF"
+		(property "Value" "100nF 50V X7R"
 			(at -0.6 -2 90)
 			(layer "B.Fab")
@@
 		)
 		(embedded_fonts no)
-		(model "${KICAD8_3DMODEL_DIR}/Capacitor_SMD.3dshapes/C_0805_2012Metric.wrl"
+		(model "${KICAD10_3DMODEL_DIR}/Capacitor_SMD.3dshapes/C_0805_2012Metric.step"
 			(offset
 				(xyz 0 0 0)
@@
 			)
 		)
-		(property "Value" "100nF"
+		(property "Value" "100nF 50V X7R"
 			(at 0 2 90)
 			(layer "B.Fab")
@@
 		)
 		(embedded_fonts no)
-		(model "${KICAD8_3DMODEL_DIR}/Capacitor_SMD.3dshapes/C_0805_2012Metric.wrl"
+		(model "${KICAD10_3DMODEL_DIR}/Capacitor_SMD.3dshapes/C_0805_2012Metric.step"
 			(offset
 				(xyz 0 0 0)
@@
 			)
 		)
-		(property "Value" "100nF"
+		(property "Value" "100nF 50V X7R"
 			(at 4.1 0.3 0)
 			(layer "B.Fab")
@@
 		)
 		(embedded_fonts no)
-		(model "${KICAD8_3DMODEL_DIR}/Capacitor_SMD.3dshapes/C_0805_2012Metric.wrl"
+		(model "${KICAD10_3DMODEL_DIR}/Capacitor_SMD.3dshapes/C_0805_2012Metric.step"
 			(offset
 				(xyz 0 0 0)
@@
 				(font
 					(size 1.27 1.27)
+					(thickness 0.15)
 				)
 				(justify mirror)
@@
 			)
 		)
-		(property "Value" "100nF"
+		(property "Value" "100nF 50V X7R"
 			(at -3.6 -1.5 90)
 			(layer "B.Fab")
@@
 		)
 		(embedded_fonts no)
-		(model "${KICAD8_3DMODEL_DIR}/Capacitor_SMD.3dshapes/C_0805_2012Metric.wrl"
+		(model "${KICAD10_3DMODEL_DIR}/Capacitor_SMD.3dshapes/C_0805_2012Metric.step"
 			(offset
 				(xyz 0 0 0)
@@
 				(font
 					(size 1.27 1.27)
+					(thickness 0.15)
 				)
 				(justify mirror)
@@
 				(font
 					(size 1.27 1.27)
+					(thickness 0.15)
 				)
 				(justify mirror)
@@
 		)
 		(embedded_fonts no)
-		(model "${KICAD8_3DMODEL_DIR}/Capacitor_SMD.3dshapes/C_0805_2012Metric.wrl"
+		(model "${KICAD10_3DMODEL_DIR}/Capacitor_SMD.3dshapes/C_0805_2012Metric.step"
 			(offset
 				(xyz 0 0 0)
@@
 		)
 		(embedded_fonts no)
-		(model "${KICAD8_3DMODEL_DIR}/Capacitor_SMD.3dshapes/C_0805_2012Metric.wrl"
+		(model "${KICAD10_3DMODEL_DIR}/Capacitor_SMD.3dshapes/C_0805_2012Metric.step"
 			(offset
 				(xyz 0 0 0)
@@
 		)
 		(embedded_fonts no)
-		(model "${KICAD8_3DMODEL_DIR}/Capacitor_SMD.3dshapes/C_0805_2012Metric.wrl"
+		(model "${KICAD10_3DMODEL_DIR}/Capacitor_SMD.3dshapes/C_0805_2012Metric.step"
 			(offset
 				(xyz 0 0 0)
@@
 				(font
 					(size 1.27 1.27)
+					(thickness 0.15)
 				)
 				(justify mirror)
@@
 				(font
 					(size 1.27 1.27)
+					(thickness 0.15)
 				)
 				(justify mirror)
@@
 		)
 		(embedded_fonts no)
-		(model "${KICAD8_3DMODEL_DIR}/Capacitor_SMD.3dshapes/C_0805_2012Metric.wrl"
+		(model "${KICAD10_3DMODEL_DIR}/Capacitor_SMD.3dshapes/C_0805_2012Metric.step"
 			(offset
 				(xyz 0 0 0)
@@
 				(font
 					(size 1.27 1.27)
+					(thickness 0.15)
 				)
 				(justify mirror)
@@
 		)
 		(embedded_fonts no)
-		(model "${KICAD8_3DMODEL_DIR}/Capacitor_SMD.3dshapes/C_0805_2012Metric.wrl"
+		(model "${KICAD10_3DMODEL_DIR}/Capacitor_SMD.3dshapes/C_0805_2012Metric.step"
 			(offset
 				(xyz 0 0 0)
@@
 		)
 		(embedded_fonts no)
-		(model "${KICAD8_3DMODEL_DIR}/Capacitor_SMD.3dshapes/C_0805_2012Metric.wrl"
+		(model "${KICAD10_3DMODEL_DIR}/Capacitor_SMD.3dshapes/C_0805_2012Metric.step"
 			(offset
 				(xyz 0 0 0)
@@
 		)
 		(embedded_fonts no)
-		(model "${KICAD8_3DMODEL_DIR}/Capacitor_SMD.3dshapes/C_0805_2012Metric.wrl"
+		(model "${KICAD10_3DMODEL_DIR}/Capacitor_SMD.3dshapes/C_0805_2012Metric.step"
 			(offset
 				(xyz 0 0 0)
@@
 				(font
 					(size 1.27 1.27)
+					(thickness 0.15)
 				)
 				(justify mirror)
@@
 				(font
 					(size 1.27 1.27)
+					(thickness 0.15)
 				)
 				(justify mirror)
@@
 		)
 		(embedded_fonts no)
-		(model "${KICAD8_3DMODEL_DIR}/Capacitor_SMD.3dshapes/C_0805_2012Metric.wrl"
+		(model "${KICAD10_3DMODEL_DIR}/Capacitor_SMD.3dshapes/C_0805_2012Metric.step"
 			(offset
 				(xyz 0 0 0)
@@
 				(font
 					(size 1.27 1.27)
+					(thickness 0.15)
 				)
 				(justify mirror)
@@
 				(font
 					(size 1.27 1.27)
+					(thickness 0.15)
 				)
 				(justify mirror)
@@
 				(font
 					(size 1.27 1.27)
+					(thickness 0.15)
 				)
 				(justify mirror)
@@
 				(font
 					(size 1.27 1.27)
+					(thickness 0.15)
 				)
 				(justify mirror)
@@
 				(font
 					(size 1.27 1.27)
+					(thickness 0.15)
 				)
 				(justify mirror)
@@
 		)
 		(embedded_fonts no)
-		(model "${KICAD8_3DMODEL_DIR}/Capacitor_SMD.3dshapes/C_0805_2012Metric.wrl"
+		(model "${KICAD10_3DMODEL_DIR}/Capacitor_SMD.3dshapes/C_0805_2012Metric.step"
 			(offset
 				(xyz 0 0 0)

Commit message: freerouting pass
Routing:
- net GND: track 0.00 -> 914.9 mm, vias 0 -> 15
- net 3v3: track 0.00 -> 315.9 mm, vias 0 -> 1
- net MCP GPB3 / L1: track 0.00 -> 171.5 mm, vias 0 -> 3
- net GPIO3 / MCP|ADC SCL: track 0.00 -> 164.6 mm, vias 0 -> 3
- net IO1 / Left Stick Y: track 0.00 -> 163.1 mm, vias 0 -> 1
- net GPIO2 / MCP|ADC SDA: track 0.00 -> 163.0 mm, vias 0 -> 4
- net MCP GPB5 / L2: track 0.00 -> 161.1 mm, vias 0 -> 3
- net IO0 / Left Stick X: track 0.00 -> 157.9 mm, vias 0 -> 1
- net IO3 / Right Stick Y: track 0.00 -> 153.2 mm, vias 0 -> 1
- net IO2 / Right Stick X: track 0.00 -> 149.3 mm, vias 0 -> 1
- net VSYS_BAT: track 0.00 -> 120.4 mm, vias 0 -> 3
- net FILTERED - IO2 / Right Stick X: track 0.00 -> 113.6 mm, vias 0 -> 2
- net GPIO16 / Left Stick: track 0.00 -> 112.1 mm
- net Net-(LS1--_(black)): track 0.00 -> 106.4 mm, vias 0 -> 1
- net FILTERED - IO3 / Right Stick Y: track 0.00 -> 105.7 mm, vias 0 -> 2
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
Commit message: no errors drc
Parts:
- moved D1 1.58 mm to (155.0, 66.0)
Routing:
- net GND: track 914.9 -> 906.4 mm, vias 15 -> 13
- net USB-VBUS: track 69.0 -> 73.9 mm, vias 1 -> 3
- net SYS_RAW: track 70.6 -> 73.7 mm, vias 0 -> 1
- net MCP GPA4 / A: track 72.2 -> 70.2 mm
- net 3v3_AUDIO: track 35.6 -> 34.0 mm
- net VSYS_BAT: track 120.4 -> 119.8 mm
- net GPIO2 / MCP|ADC SDA: track 163.0 -> 162.5 mm
- net MCP GPB6 / R2: track 104.2 -> 103.7 mm

Commit message: clean up tracks
Routing:
- net IO1 / Left Stick Y: track 163.1 -> 159.4 mm
- net IO0 / Left Stick X: track 157.9 -> 154.3 mm
- net GND: track 906.4 -> 903.9 mm
- net MCP GPA1 / DPAD - DOWN: track 103.5 -> 101.0 mm
- net 3v3: track 315.9 -> 317.8 mm
- net FILTERED - IO1 / Left Stick Y: track 76.8 -> 78.2 mm
- net GPIO11 / MAX LRC: track 34.6 -> 35.4 mm
- net DAC_R: track 44.0 -> 43.3 mm
- net GPIO14 / SD SCK: track 85.4 -> 84.7 mm
- net GPIO2 / MCP|ADC SDA: track 162.5 -> 163.1 mm
- net FILTERED - IO0 / Left Stick X: track 63.5 -> 63.0 mm
- net GPIO16 / Left Stick: track 112.1 -> 112.6 mm

Commit message: fix a bunch of footprints and routing
Parts:
- FB1, FB4, FB5: footprint PCM_SparkFun-Capacitor:C_0603_1608Metric -> Ferrite_THT:LairdTech_28C0236-0JW-10
- moved FB4 12.4 mm to (137.7, 90.3)
- moved FB1 11.0 mm to (105.4, 131.9), turned to 0 degrees
- moved FB5 6.71 mm to (162.9, 85.6)
- moved C16 0.15 mm to (154.3, 102.7)
Connections:
- A2 pad 33: AGND -> GND
- A2 pad 34: GPIO28 / VOLUME POT -> unconnected-(A2-GPIO28_ADC2-Pad34)
- C15 pad 2: GND -> 3v3_AUDIO
- C17 pad 2: GND -> 3v3_AUDIO
- C41 pad 2: GND -> 3v3_AUDIO
Routing:
- net 3v3_AUDIO: track 34.0 -> 56.3 mm, vias 2 -> 3
- net 3v3: track 317.8 -> 337.5 mm, vias 1 -> 2
- net GND: track 903.9 -> 920.5 mm
- net 3v3_ADC: track 3.83 -> 11.0 mm, vias 0 -> 2
- net VSYS_BAT: track 119.8 -> 113.4 mm
- net AMP_VDD: track 77.5 -> 83.0 mm, vias 4 -> 6
- net GPIO28 / VOLUME POT: track 0.80 -> 0.00 mm
- net AGND: track 0.80 -> 0.00 mm
- net (no net): track 0.00 -> 0.80 mm

Commit message: fix up design and parts
Parts:
- removed SW1: SW_Nidec_CAS-120A1, Button_Switch_SMD:Nidec_Copal_CAS-120A
- added SW19: SPDT_Slide_PTH_11.6x4.0mm, PCM_SparkFun-Switch:Slide_SPDT_PTH_11.6x4.0mm, F.Cu at (132.7, 61.4)
- D1: footprint PCM_SparkFun-Sensor:Sensirion_DFN-4_1.5x1.5mm_P0.8mm_SHT4x_NoCentralPad -> Diode_SMD:Nexperia_CFP3_SOD-123W
- Q1: footprint Package_TO_SOT_THT:TO-92 -> Package_TO_SOT_SMD:SOT-23
- U1: value MCP73833_MSOP -> MCP73833-FCI/UN
- moved D1 3.13 mm to (158.0, 66.9), turned to -90 degrees
- moved Q1 2.15 mm to (193.7, 63.0), turned to 0 degrees
Connections:
- A2 pad 33: GND -> unconnected-(A2-AGND-Pad33)
- D1 pad 1: SYS_RAW -> USB-VBUS
- D1 pad 2: USB-VBUS -> SYS_RAW
- Q1 pad 2: SYS_RAW -> BAT+
- Q1 pad 3: BAT+ -> SYS_RAW
Routing:
- net GND: track 920.5 -> 900.2 mm
- net BAT+: track 35.0 -> 28.2 mm, vias 0 -> 1
- net USB-VBUS: track 73.9 -> 79.4 mm, vias 3 -> 6
- net VSYS_BAT: track 113.4 -> 110.6 mm, vias 3 -> 2
- net SYS_RAW: track 73.7 -> 75.7 mm
- net unconnected-(A2-AGND-Pad33): track 0.00 -> 0.80 mm
- net (no net): track 0.80 -> 0.00 mm
- net Net-(D2-K): track 15.8 -> 16.4 mm
