File: microconsole_hardware/mc_hw/battery.kicad_sch (KiCad schematic)
At the start: 19 parts, among them J1 USB_C_Receptacle_USB2.0_16P, Q1 Q_PMOS_GSD, SW1 SW_Nidec_CAS-120A1, U1 MCP73833_MSOP, U2 S2B-PH-K-S

Commit message: fix up everything,
Parts:
- Q1: footprint (none) -> Package_TO_SOT_THT:TO-92
Changed lines of the file:
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@@
 		)
 		(instances
-			(project "mc_hw"
+			(project "top"
 				(path "/3433afdc-e53a-48bd-a2b1-9fdee73e8b40/2e88eeda-748f-4d75-b88b-5acda3278369"
 					(reference "R6")
@@
 		)
 		(instances
-			(project "mc_hw"
+			(project "top"
 				(path "/3433afdc-e53a-48bd-a2b1-9fdee73e8b40/2e88eeda-748f-4d75-b88b-5acda3278369"
 					(reference "R5")
@@
 		)
 		(instances
-			(project "mc_hw"
+			(project "top"
 				(path "/3433afdc-e53a-48bd-a2b1-9fdee73e8b40/2e88eeda-748f-4d75-b88b-5acda3278369"
 					(reference "R7")
@@
 		)
 		(instances
-			(project "mc_hw"
+			(project "top"
 				(path "/3433afdc-e53a-48bd-a2b1-9fdee73e8b40/2e88eeda-748f-4d75-b88b-5acda3278369"
 					(reference "C1")
@@
 		)
 		(instances
-			(project "mc_hw"
+			(project "top"
 				(path "/3433afdc-e53a-48bd-a2b1-9fdee73e8b40/2e88eeda-748f-4d75-b88b-5acda3278369"
 					(reference "U1")
@@
 		)
 		(instances
-			(project "mc_hw"
+			(project "top"
 				(path "/3433afdc-e53a-48bd-a2b1-9fdee73e8b40/2e88eeda-748f-4d75-b88b-5acda3278369"
 					(reference "J1")
@@
 		)
 		(instances
-			(project "mc_hw"
+			(project "top"
 				(path "/3433afdc-e53a-48bd-a2b1-9fdee73e8b40/2e88eeda-748f-4d75-b88b-5acda3278369"
 					(reference "U2")
@@
 		)
 		(instances
-			(project "mc_hw"
+			(project "top"
 				(path "/3433afdc-e53a-48bd-a2b1-9fdee73e8b40/2e88eeda-748f-4d75-b88b-5acda3278369"
 					(reference "D1")
@@
 		)
 		(instances
-			(project "mc_hw"
+			(project "top"
 				(path "/3433afdc-e53a-48bd-a2b1-9fdee73e8b40/2e88eeda-748f-4d75-b88b-5acda3278369"
 					(reference "R9")
@@
 			)
 		)
-		(property "Footprint" ""
+		(property "Footprint" "Package_TO_SOT_THT:TO-92"
 			(at 123.19 60.96 0)
 			(hide yes)
@@
 		)
 		(instances
-			(project "mc_hw"
+			(project "top"
 				(path "/3433afdc-e53a-48bd-a2b1-9fdee73e8b40/2e88eeda-748f-4d75-b88b-5acda3278369"
 					(reference "Q1")
@@
 		)
 		(instances
-			(project "mc_hw"
+			(project "top"
 				(path "/3433afdc-e53a-48bd-a2b1-9fdee73e8b40/2e88eeda-748f-4d75-b88b-5acda3278369"
 					(reference "SW1")
@@
 		)
 		(instances
-			(project "mc_hw"
+			(project "top"
 				(path "/3433afdc-e53a-48bd-a2b1-9fdee73e8b40/2e88eeda-748f-4d75-b88b-5acda3278369"
 					(reference "D4")
@@
 		)
 		(instances
-			(project "mc_hw"
+			(project "top"
 				(path "/3433afdc-e53a-48bd-a2b1-9fdee73e8b40/2e88eeda-748f-4d75-b88b-5acda3278369"
 					(reference "R8")
@@
 		)
 		(instances
-			(project "mc_hw"
+			(project "top"
 				(path "/3433afdc-e53a-48bd-a2b1-9fdee73e8b40/2e88eeda-748f-4d75-b88b-5acda3278369"
 					(reference "R10")
@@
 		)
 		(instances
-			(project "mc_hw"
+			(project "top"
 				(path "/3433afdc-e53a-48bd-a2b1-9fdee73e8b40/2e88eeda-748f-4d75-b88b-5acda3278369"
 					(reference "C2")
@@
 		)
 		(instances
-			(project "mc_hw"
+			(project "top"
 				(path "/3433afdc-e53a-48bd-a2b1-9fdee73e8b40/2e88eeda-748f-4d75-b88b-5acda3278369"
 					(reference "D2")
@@
 		)
 		(instances
-			(project "mc_hw"
+			(project "top"
 				(path "/3433afdc-e53a-48bd-a2b1-9fdee73e8b40/2e88eeda-748f-4d75-b88b-5acda3278369"
 					(reference "D3")
@@
 		)
 		(instances
-			(project "mc_hw"
+			(project "top"
 				(path "/3433afdc-e53a-48bd-a2b1-9fdee73e8b40/2e88eeda-748f-4d75-b88b-5acda3278369"
 					(reference "R3")
@@
 		)
 		(instances
-			(project "mc_hw"
+			(project "top"
 				(path "/3433afdc-e53a-48bd-a2b1-9fdee73e8b40/2e88eeda-748f-4d75-b88b-5acda3278369"
 					(reference "R4")

Commit message: fix up design and parts
Parts:
- removed SW1: SW_Nidec_CAS-120A1, Button_Switch_SMD:Nidec_Copal_CAS-120A, symbol Switch:SW_Nidec_CAS-120A1
- added SW19: SPDT_Slide_PTH_11.6x4.0mm, PCM_SparkFun-Switch:Slide_SPDT_PTH_11.6x4.0mm, symbol PCM_SparkFun-Switch:SPDT_Slide_PTH_11.6x4.0mm
- D1: footprint PCM_SparkFun-Sensor:Sensirion_DFN-4_1.5x1.5mm_P0.8mm_SHT4x_NoCentralPad -> Diode_SMD:Nexperia_CFP3_SOD-123W
- J1: symbol Connector:USB_C_Receptacle_USB2.0_16P -> project_parts:USB_C_Receptacle_USB2.0_16P
- Q1: footprint Package_TO_SOT_THT:TO-92 -> Package_TO_SOT_SMD:SOT-23
- U1: value MCP73833_MSOP -> MCP73833-FCI/UN
Connections:
- net BAT+: now also Q1.2 (S); no longer Q1.3 (D)
- net SYS_RAW: now also D1.2 (A), Q1.3 (D), SW19.2 (B); no longer D1.1 (K), Q1.2 (S)
- net VDD: now also D1.1 (K); no longer D1.2 (A)
- net VSYS_BAT: now also SW19.1 (A)
Other:
- moved on the sheet: R5

Commit message: fix up power and parts
Parts:
- added Q2: DMP2035U-7, Package_TO_SOT_SMD:SOT-23, symbol Transistor_FET:Q_PMOS_GSD
- added R31: 100k, PCM_SparkFun-Resistor:R_0603_1608Metric, symbol PCM_SparkFun-Resistor:0.47_0603
- Q1: value Q_PMOS_GSD -> DMP2035U-7
Connections:
- net BAT+: now also C2.1, Q1.3 (D); no longer Q1.2 (S)
- net GND: now also SW19.1 (A), U2.2
- net SYS_RAW: now also D1.1 (K), Q1.2 (S), Q2.2 (S), R31.1; no longer D1.2 (A), Q1.3 (D), SW19.2 (B)
- net VDD: now also D1.2 (A); no longer D1.1 (K)
- net VSYS_BAT: now also Q2.3 (D); no longer SW19.1 (A)
- new net PWR_SW_GATE: Q2.1 (G), R31.2, SW19.2 (B)
Other:
- moved on the sheet: D1, R5, SW19

Commit message: fix up some problems. still net battery protection and audio gain protection
Parts:
- D1: value D_Schottky -> PMEG40T30ER Schottky
Changed lines of the file:
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@@
 			)
 		)
-		(property "Value" "D_Schottky"
+		(property "Value" "PMEG40T30ER Schottky"
 			(at 120.9675 34.29 0)
 			(show_name no)

Commit message: eh more fixes
Parts:
- R9: value 2k -> 3.32k
Changed lines of the file:
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@@
 			)
 		)
-		(property "Value" "2k"
+		(property "Value" "3.32k"
 			(at 227.33 60.9599 90)
 			(show_name no)

Commit message: fixup
Parts:
- added D5: BAT54C, Package_TO_SOT_SMD:SOT-23, symbol Diode:BAT54C
Connections:
- net VDD: now also D5.1; no longer Q1.1 (G), R5.1
- new net: D5.3, Q1.1 (G), R5.1
- new net PICO_VBUS: D5.2
Other:
- moved on the sheet: Q1, R5

Commit message: fix up
Parts:
- D1: footprint Diode_SMD:Nexperia_CFP3_SOD-123W -> (none)
- D2, D3, D4: footprint PCM_SparkFun-Resistor:R_0603_1608Metric -> (none)
- Q1, Q2: footprint Package_TO_SOT_SMD:SOT-23 -> (none)
Changed lines of the file:
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@@
 			)
 		)
-		(property "Footprint" "Diode_SMD:Nexperia_CFP3_SOD-123W"
+		(property "Footprint" ""
 			(at 120.65 38.1 0)
 			(hide yes)
@@
 			)
 		)
-		(property "Datasheet" "https://assets.nexperia.com/documents/data-sheet/PMEG40T30ER.pdf"
+		(property "Datasheet" ""
 			(at 120.65 38.1 0)
 			(hide yes)
@@
 			)
 		)
-		(property "Datasheet" "https://www.mouser.com/datasheet/3/282/1/22005b.pdf"
+		(property "Datasheet" "https://ww1.microchip.com/downloads/en/DeviceDoc/22005b.pdf"
 			(at 212.09 50.8 0)
 			(hide yes)
@@
 			)
 		)
-		(property "Footprint" "Package_TO_SOT_SMD:SOT-23"
+		(property "Footprint" ""
 			(at 137.16 109.22 0)
 			(hide yes)
@@
 			)
 		)
-		(property "Footprint" "PCM_SparkFun-Resistor:R_0603_1608Metric"
+		(property "Footprint" ""
 			(at 191.77 44.45 0)
 			(hide yes)
@@
 			)
 		)
-		(property "Footprint" "PCM_SparkFun-Resistor:R_0603_1608Metric"
+		(property "Footprint" ""
 			(at 157.48 44.45 0)
 			(hide yes)
@@
 			)
 		)
-		(property "Footprint" "PCM_SparkFun-Resistor:R_0603_1608Metric"
+		(property "Footprint" ""
 			(at 173.99 44.45 0)
 			(hide yes)
@@
 			)
 		)
-		(property "Footprint" "Package_TO_SOT_SMD:SOT-23"
+		(property "Footprint" ""
 			(at 129.54 59.69 0)
 			(hide yes)
