File: microconsole_hardware/mc_hw/audio.kicad_sch (KiCad schematic)
At the start: 47 parts, among them U5 PCM5102APWR, U6 PAM8302AADCR, U7 PAM8406DR

Commit message: second fix
Parts:
- FB4: MPN (none) -> MPZ1608S601ATA00; Manufacturer (none) -> TDK
Changed lines of the file:
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@@
+			)
+		)
+		(property "MPN" "MPZ1608S601ATA00"
+			(at 241.3 44.45 90)
+			(hide yes)
+			(show_name no)
+			(do_not_autoplace no)
+			(effects
+				(font
+					(size 1.27 1.27)
+				)
+			)
+		)
+		(property "Manufacturer" "TDK"
+			(at 241.3 44.45 90)
+			(hide yes)
+			(show_name no)
+			(do_not_autoplace no)
+			(effects
+				(font
+					(size 1.27 1.27)
+				)
 			)
 		)

Commit message: fix up bom
Parts:
- C18, C19: MPN (none) -> C0805C222J5GECTU; Manufacturer (none) -> KEMET
- C22, C28: MPN (none) -> GRM21BR71C225KA12L; Manufacturer (none) -> Murata Electronics
- C23: MPN (none) -> C0805C333K5RECAUTO; Manufacturer (none) -> KEMET
- C31, C59: MPN (none) -> C2012X7R1H224K125AA; Manufacturer (none) -> TDK
- C32, C72: MPN (none) -> C2012X7R1H474K125AB; Manufacturer (none) -> TDK
- C34, C37, C39, C73: MPN (none) -> GRM21BR71C105KA01L; Manufacturer (none) -> Murata Electronics

Commit message: bom cleanup
Parts:
- C14, C16, C33, C36, C40, C44: Tolerance (none) -> 10%; Voltage (none) -> 50V
- C15, C17, C29, C35, C38, C41: Tolerance (none) -> 10%; Voltage (none) -> 10V
- C18, C19: PROD_ID CAP-11624 -> (none); Tolerance 20% -> 5%; Voltage 25V -> 50V
- C22, C28, C34, C37, C39, C73: PROD_ID CAP-11624 -> (none); Tolerance 20% -> 10%; Voltage 25V -> 16V
- C23, C31, C32, C59, C72: PROD_ID CAP-11624 -> (none); Tolerance 20% -> 10%; Voltage 25V -> 50V

Commit message: dnp
Parts:
- LS1, LS2, LS3, RV1: now not fitted
Changed lines of the file:
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@@
 		(on_board yes)
 		(in_pos_files yes)
-		(dnp no)
+		(dnp yes)
 		(property "Reference" "LS1"
 			(at 121.666 93.218 90)
@@
 		(on_board yes)
 		(in_pos_files yes)
-		(dnp no)
+		(dnp yes)
 		(fields_autoplaced yes)
 		(property "Reference" "LS2"
@@
 		(on_board yes)
 		(in_pos_files yes)
-		(dnp no)
+		(dnp yes)
 		(property "Reference" "LS3"
 			(at 176.53 93.98 0)
@@
 		(on_board yes)
 		(in_pos_files yes)
-		(dnp no)
+		(dnp yes)
 		(fields_autoplaced yes)
 		(property "Reference" "RV1"
