File: microconsole_hardware/mc_hw/top_withnets.kicad_pcb (KiCad board)
At the start: 2 copper layers, 161 x 96 mm, 115 parts, among them J2 USB_C_Receptacle, Q1 DMP2035U-7, Q2 DMP2035U-7, SW10 TL3301NF160QG, SW11 TL3301NF160QG, SW12 TL3301NF160QG, SW13 TL3301NF160QG, SW14 TL3301NF160QG, SW15 TL3301NF160QG, SW16 FJH10K-S2, SW17 FJH10K-S2, SW19 SPDT_Slide_PTH_11.6x4.0mm, SW2 TL3301NF160QG, SW3 TL3301NF160QG, SW4 TL3301NF160QG, SW5 TL3301NF160QG, SW6 TL3301NF160QG, SW7 TL3301NF160QG, SW8 TL3301NF160QG, SW9 TL3301NF160QG, U1 MCP73833-FCI/UN, U2 S2B-PH-K-S, U3 MCP23017-E/SO, U4 ADS7828E/2K5, U5 PCM5102APWR, U6 PAM8302AADCR, U7 PAM8406DR

Commit message: new pcb
Routing:
- net PICO_VBUS: track 28.9 -> 224.7 mm, vias 2 -> 9
- net GPIO2 / MCP|ADC SDA: track 367.7 -> 229.2 mm, vias 6 -> 8
- net GPIO7 / LCD MOSI: track 30.2 -> 136.0 mm, vias 0 -> 8
- net GPIO5 / LCD CS: track 30.2 -> 111.3 mm, vias 0 -> 3
- net GPIO6 / LCD SCK: track 35.9 -> 101.5 mm, vias 0 -> 3
- net GPIO8 / LCD RESET: track 40.4 -> 104.5 mm, vias 0 -> 3
- net GPIO9 / LCD DC: track 38.6 -> 100.6 mm, vias 0 -> 3
- net Net-(LS1-+_(red)): track 103.5 -> 162.8 mm, vias 1 -> 7
- net Net-(LS1--_(black)): track 106.4 -> 160.1 mm, vias 1 -> 7
- net GPIO4 / LCD MISO: track 37.6 -> 88.7 mm, vias 0 -> 3
- net GPIO20 / MAX DIN: track 50.3 -> 87.1 mm, vias 1 -> 3
- net GPIO3 / MCP|ADC SCL: track 164.6 -> 199.6 mm, vias 3 -> 5
- net Net-(Q1-G): track 92.6 -> 68.0 mm, vias 5 -> 2
- net VSYS_BAT: track 253.3 -> 270.9 mm, vias 12 -> 8
- net MCP GPB3 / L1: track 162.3 -> 178.1 mm
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Other:
- outline, holes or cut-outs redrawn

Commit message: new pcb
Parts:
- moved R29 0.34 mm to (165.8, 95.6)
Routing:
- net GPIO2 / MCP|ADC SDA: track 229.2 -> 219.1 mm, vias 8 -> 6
- net GND: track 955.7 -> 946.4 mm, vias 19 -> 20
- net USB-VBUS: track 85.3 -> 89.1 mm
- net Net-(LS3-+_(red)): track 48.6 -> 52.2 mm
- net Net-(LS3--_(black)): track 56.6 -> 53.3 mm
- net Net-(LS1--_(black)): track 160.1 -> 163.0 mm
- net GPIO4 / LCD MISO: track 88.7 -> 90.6 mm
- net PICO_VBUS: track 224.7 -> 223.1 mm
- net MCP GPB3 / L1: track 178.1 -> 176.5 mm
- net GPIO17 / Right Stick: track 121.2 -> 122.5 mm
- net FILTERED - IO2 / Right Stick X: track 109.8 -> 108.6 mm, vias 2 -> 4
- net 3v3: track 360.0 -> 361.0 mm
- net DAC_R: track 39.4 -> 38.4 mm
- net Net-(LS2-+): track 28.5 -> 29.4 mm
- net Net-(LS1-+_(red)): track 162.8 -> 163.6 mm
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