File: microconsole_hardware/mc_hw/joysticks/buttons.kicad_sch (KiCad schematic)
At the start: 32 parts, among them SW17 Joystick, SW18 Joystick, SW33 TL3301NF160QG, SW34 TL3301NF160QG, SW35 TL3301NF160QG, SW36 TL3301NF160QG, SW37 TL3301NF160QG, SW38 TL3301NF160QG, SW39 TL3301NF160QG, SW40 TL3301NF160QG, SW41 TL3301NF160QG, SW42 TL3301NF160QG, SW43 TL3301NF160QG, SW44 TL3301NF160QG, SW45 TL3301NF160QG, SW46 TL3301NF160QG, U15 ADS7828E/2K5, U16 MCP23017-E/SO

Commit message: update
Parts:
- added FB1: FerriteBead_Small, PCM_SparkFun-Capacitor:C_0603_1608Metric, symbol Device:FerriteBead_Small
Connections:
- net 3v3: now also FB1.1
- net 3v3_ADC: now also FB1.2
Changed lines of the file:
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@@
 	(wire
 		(pts
+			(xy 273.05 49.53) (xy 271.78 49.53)
+		)
+		(stroke
+			(width 0)
+			(type default)
+		)
+	)
+	(wire
+		(pts
 			(xy 77.47 165.1) (xy 77.47 160.02)
 		)
@@
 	(wire
 		(pts
+			(xy 265.43 49.53) (xy 266.7 49.53)
+		)
+		(stroke
+			(width 0)
+			(type default)
+		)
+	)
+	(wire
+		(pts
 			(xy 229.87 101.6) (xy 232.41 101.6)
 		)
@@
 		)
 	)
+	(global_label "3v3_ADC"
+		(shape input)
+		(at 218.44 38.1 0)
+		(fields_autoplaced yes)
+		(effects
+			(font
+				(size 1.27 1.27)
+			)
+			(justify left)
+		)
+		(property "Intersheetrefs" "${INTERSHEET_REFS}"
+			(at 229.408 38.1 0)
+			(hide yes)
+			(show_name no)
+			(do_not_autoplace no)
+			(effects
+				(font
+					(size 1.27 1.27)
+				)
+				(justify left)
+			)
+		)
+	)
 	(global_label "GND"
 		(shape input)
@@
 		)
 	)
-	(global_label "3v3_ADC"
+	(global_label "3v3"
 		(shape input)
-		(at 218.44 38.1 0)
+		(at 273.05 49.53 0)
 		(fields_autoplaced yes)
 		(effects
@@
 		)
 		(property "Intersheetrefs" "${INTERSHEET_REFS}"
-			(at 229.408 38.1 0)
+			(at 279.4218 49.53 0)
 			(hide yes)
 			(show_name no)
@@
 		)
 	)
+	(global_label "3v3_ADC"
+		(shape input)
+		(at 265.43 49.53 180)
+		(fields_autoplaced yes)
+		(effects
+			(font
+				(size 1.27 1.27)
+			)
+			(justify right)
+		)
+		(property "Intersheetrefs" "${INTERSHEET_REFS}"
+			(at 254.462 49.53 0)
+			(hide yes)
+			(show_name no)
+			(do_not_autoplace no)
+			(effects
+				(font
+					(size 1.27 1.27)
+				)
+				(justify right)
+			)
+		)
+	)
 	(global_label "MCP GPB3 {slash} L1"
 		(shape input)
@@
 					(unit 1)
 				)
+			)
+		)
+	)
+	(symbol
+		(lib_id "Device:FerriteBead_Small")
+		(at 269.24 49.53 270)
+		(unit 1)
+		(body_style 1)
+		(exclude_from_sim no)
+		(in_bom yes)
+		(on_board yes)
+		(in_pos_files yes)
+		(dnp no)
+		(fields_autoplaced yes)
+		(property "Reference" "FB1"
+			(at 269.2781 43.18 90)
+			(show_name no)
+			(do_not_autoplace no)
+			(effects
+				(font
+					(size 1.27 1.27)
+				)
+			)
+		)
+		(property "Value" "FerriteBead_Small"
+			(at 269.2781 45.72 90)
+			(show_name no)
+			(do_not_autoplace no)
+			(effects
+				(font
+					(size 1.27 1.27)
+				)
+			)
+		)
+		(property "Footprint" "PCM_SparkFun-Capacitor:C_0603_1608Metric"
+			(at 269.24 47.752 90)
+			(hide yes)
+			(show_name no)
+			(do_not_autoplace no)
+			(effects
+				(font
+					(size 1.27 1.27)
+				)
+			)
+		)
+		(property "Datasheet" ""
+			(at 269.24 49.53 0)
+			(hide yes)
+			(show_name no)
+			(do_not_autoplace no)
+			(effects
+				(font
+					(size 1.27 1.27)
+				)
+			)
+		)
+		(property "Description" "Ferrite bead, small symbol"
+			(at 269.24 49.53 0)
+			(hide yes)
+			(show_name no)
+			(do_not_autoplace no)
+			(effects
+				(font
+					(size 1.27 1.27)
+				)
+			)
+		)
+		(pin "2"
+		)
+		(pin "1"
+		)
+		(instances
+			(project "mc_hw"
+				(path "/719302af-dc57-4543-bdcd-0eb891c4def3"
+					(reference "FB1")
+					(unit 1)
+				)
