File: microconsole_hardware/catBUS_MEOW/catBUS_MEOW.kicad_pcb (KiCad board)
At the start: 2 copper layers, 33 x 44.2 mm, 43 parts, among them J1 Conn_01x10, J2 Conn_01x10, U5 PCM5102APWR, U6 PAM8302AADCR, U7 PAM8406DR

Commit message: a
Parts:
- moved C35 0.09 mm to (211.6, 137.5)
Routing:
- net VSYS_BAT: track 77.9 -> 73.1 mm
- net GND: track 205.0 -> 201.1 mm
- net Net-(U5-LDOO): track 10.2 -> 7.69 mm
- net DAC_R: track 42.9 -> 41.2 mm
- net DAC_L: track 40.0 -> 39.2 mm
Other:
- outline, holes or cut-outs redrawn
